Commit message: update

File: urdf/diffbot.materials.xacro (robot description, xacro)
@@ -6,26 +6,26 @@
 <robot>
   <material name="black">
-    <color rgba="0.0 0.0 0.0 1.0"/>
+    <color rgba="0.0 0.0 0.0 1.0" />
   </material>
   <material name="blue">
-    <color rgba="0.0 0.0 0.8 1.0"/>
+    <color rgba="0.0 0.0 0.8 1.0" />
   </material>
   <material name="green">
-    <color rgba="0.0 0.8 0.0 1.0"/>
+    <color rgba="0.0 0.8 0.0 1.0" />
   </material>
   <material name="grey">
-    <color rgba="0.2 0.2 0.2 1.0"/>
+    <color rgba="0.2 0.2 0.2 1.0" />
   </material>
   <material name="orange">
-    <color rgba="${255/255} ${108/255} ${10/255} 1.0"/>
+    <color rgba="${255/255} ${108/255} ${10/255} 1.0" />
   </material>
   <material name="brown">
-    <color rgba="${222/255} ${207/255} ${195/255} 1.0"/>
+    <color rgba="${222/255} ${207/255} ${195/255} 1.0" />
   </material>
   <material name="red">
-    <color rgba="0.8 0.0 0.0 1.0"/>
+    <color rgba="0.8 0.0 0.0 1.0" />
   </material>
   <material name="white">
-    <color rgba="1.0 1.0 1.0 1.0"/>
+    <color rgba="1.0 1.0 1.0 1.0" />
   </material>
 </robot>

File: urdf/diffbot_description.urdf.xacro (robot description, xacro)
@@ -3,5 +3,5 @@
   <xacro:macro name="diffbot" params="prefix">
     <!-- Constants for robot dimensions -->
-    <xacro:property name="PI" value="3.1415926535897931"/>
+    <xacro:property name="PI" value="3.1415926535897931" />
     <xacro:property name="base_mass" value="0.3" /> <!-- arbitrary value for base mass -->
     <xacro:property name="base_width" value="0.25" /> <!-- Updated wheel spacing to 25cm -->
@@ -11,50 +11,54 @@
     <xacro:property name="wheel_len" value="0.020" />
     <xacro:property name="wheel_radius" value="0.0625" />
-    <xacro:property name="caster_wheel_mass" value="0.1" /> <!-- arbitrary value for caster wheel mass -->
+    <xacro:property name="caster_wheel_mass" value="0.1" /> <!-- arbitrary value for caster wheel
+    mass -->
     <xacro:property name="caster_wheel_radius" value="0.04" />
-    <xacro:property name="z_offset" value="-${base_height/2}" /> <!-- Space btw top of beam and the each joint -->
+    <xacro:property name="z_offset" value="-${base_height/2}" /> <!-- Space btw top of beam and the
+    each joint -->
     <!-- dummy link - used for ros2 control so it stops complaining? -->
     <link name="${prefix}dummy">
     </link>
     <joint name="${prefix}dummy_joint" type="fixed">
-      <parent link="${prefix}dummy"/>
-      <child link="${prefix}base_link"/>
+      <parent link="${prefix}dummy" />
+      <child link="${prefix}base_link" />
     </joint>
     <!-- Base Link -->
     <link name="${prefix}base_link">
       <collision>
-        <origin xyz="0 0 0" rpy="0 0 0"/>
-        <geometry>
-          <box size="${base_length} ${base_width} ${base_height}"/> <!-- Updated base dimensions -->
-        </geometry>
-      </collision>
-      <visual>
-        <origin xyz="0 0 ${base_height/2}" rpy="0 0 0"/>
-        <geometry>
-          <box size="${base_length} ${base_width} ${base_height}"/> <!-- Updated base dimensions -->
-        </geometry>
-        <material name="orange"/>
-      </visual>
-      <inertial>
-        <origin xyz="0 0 0" rpy="0 0 0"/>
-        <mass value="${base_mass}"/>
-        <inertia
-          ixx="${base_mass / 12.0 * (base_length*base_length + base_height*base_height)}" ixy="0.0" ixz="0.0"
+        <origin xyz="0 0 0" rpy="0 0 0" />
+        <geometry>
+          <box size="${base_length} ${base_width} ${base_height}" /> <!-- Updated base dimensions -->
+        </geometry>
+      </collision>
+      <visual>
+        <origin xyz="0 0 ${base_height/2}" rpy="0 0 0" />
+        <geometry>
+          <box size="${base_length} ${base_width} ${base_height}" /> <!-- Updated base dimensions -->
+        </geometry>
+        <material name="orange" />
+      </visual>
+      <inertial>
+        <origin xyz="0 0 0" rpy="0 0 0" />
+        <mass value="${base_mass}" />
+        <inertia
+          ixx="${base_mass / 12.0 * (base_length*base_length + base_height*base_height)}" ixy="0.0"
+          ixz="0.0"
           iyy="${base_mass / 12.0 * (base_height*base_height + base_width*base_width)}" iyz="0.0"
-          izz="${base_mass / 12.0 * (base_width*base_width + base_length*base_length)}"/>
+          izz="${base_mass / 12.0 * (base_width*base_width + base_length*base_length)}" />
       </inertial>
     </link>
     <joint name="${prefix}left_wheel_joint" type="continuous">
-      <parent link="${prefix}base_link"/>
-      <child link="${prefix}left_wheel"/>
-      <origin xyz="${base_length/2} 0 ${z_offset}" rpy="0 0 0"/> <!-- Updated wheel position -->
-      <axis xyz="0 1 0"/>
-      <dynamics damping="0.2"/>
-    </joint>
-    <!-- BASE_FOOTPRINT LINK (Used for SLAM: Should be oin the ground beneath the robo like the shadow) -->
+      <parent link="${prefix}base_link" />
+      <child link="${prefix}left_wheel" />
+      <origin xyz="${base_length/2} 0 ${z_offset}" rpy="0 0 0" /> <!-- Updated wheel position -->
+      <axis xyz="0 1 0" />
+      <dynamics damping="0.2" />
+    </joint>
+    <!-- BASE_FOOTPRINT LINK (Used for SLAM: Should be oin the ground beneath the robo like the
+    shadow) -->
     <joint name="${prefix}base_footprint_joint" type="fixed">
-      <parent link="${prefix}base_link"/>
-      <child link="${prefix}base_footprint"/>
-      <origin xyz="0 0 0" rpy="0 0 0"/>
+      <parent link="${prefix}base_link" />
+      <child link="${prefix}base_footprint" />
+      <origin xyz="0 0 0" rpy="0 0 0" />
     </joint>
     <link name="${prefix}base_footprint">
@@ -63,147 +67,147 @@
     <link name="${prefix}left_wheel">
       <collision>
-        <origin xyz="0 0 0" rpy="${PI/2} 0 0"/>
-        <geometry>
-          <cylinder length="${wheel_len}" radius="${wheel_radius}"/>
-        </geometry>
-      </collision>
-      <visual>
-        <origin xyz="0 0 0" rpy="${PI/2} 0 0"/>
-        <geometry>
-          <cylinder length="${wheel_len}" radius="${wheel_radius}"/>
-        </geometry>
-        <material name="black"/>
-      </visual>
-      <inertial>
-        <origin xyz="0 0 0" rpy="${PI/2} 0 0"/>
-        <mass value="${wheel_mass}"/>
+        <origin xyz="0 0 0" rpy="${PI/2} 0 0" />
+        <geometry>
+          <cylinder length="${wheel_len}" radius="${wheel_radius}" />
+        </geometry>
+      </collision>
+      <visual>
+        <origin xyz="0 0 0" rpy="${PI/2} 0 0" />
+        <geometry>
+          <cylinder length="${wheel_len}" radius="${wheel_radius}" />
+        </geometry>
+        <material name="black" />
+      </visual>
+      <inertial>
+        <origin xyz="0 0 0" rpy="${PI/2} 0 0" />
+        <mass value="${wheel_mass}" />
         <inertia
           ixx="${wheel_mass / 12.0 * (3*wheel_radius + wheel_len*wheel_len)}" ixy="0.0" ixz="0.0"
           iyy="${wheel_mass / 12.0 * wheel_radius*wheel_radius}" iyz="0.0"
-          izz="${wheel_mass / 12.0 * wheel_radius*wheel_radius}"/>
+          izz="${wheel_mass / 12.0 * wheel_radius*wheel_radius}" />
       </inertial>
     </link>
     <joint name="${prefix}right_wheel_joint" type="continuous">
-      <parent link="${prefix}base_link"/>
-      <child link="${prefix}right_wheel"/>
-      <origin xyz="${base_length/2} 0 ${z_offset}" rpy="0 0 0"/> <!-- Updated wheel position -->
-      <axis xyz="0 -1 0"/>
-      <dynamics damping="0.2"/>
+      <parent link="${prefix}base_link" />
+      <child link="${prefix}right_wheel" />
+      <origin xyz="${base_length/2} 0 ${z_offset}" rpy="0 0 0" /> <!-- Updated wheel position -->
+      <axis xyz="0 -1 0" />
+      <dynamics damping="0.2" />
     </joint>
     <!-- right wheel Link -->
     <link name="${prefix}right_wheel">
       <collision>
-        <origin xyz="0 0 0" rpy="${PI/2} 0 0"/>
-        <geometry>
-          <cylinder length="${wheel_len}" radius="${wheel_radius}"/>
-        </geometry>
-      </collision>
-      <visual>
-        <origin xyz="0 0 0" rpy="${PI/2} 0 0"/>
-        <geometry>
-          <cylinder length="${wheel_len}" radius="${wheel_radius}"/>
-        </geometry>
-        <material name="black"/>
-      </visual>
-      <inertial>
-        <origin xyz="0 0 0" rpy="${PI/2} 0 0"/>
-        <mass value="${wheel_mass}"/>
+        <origin xyz="0 0 0" rpy="${PI/2} 0 0" />
+        <geometry>
+          <cylinder length="${wheel_len}" radius="${wheel_radius}" />
+        </geometry>
+      </collision>
+      <visual>
+        <origin xyz="0 0 0" rpy="${PI/2} 0 0" />
+        <geometry>
+          <cylinder length="${wheel_len}" radius="${wheel_radius}" />
+        </geometry>
+        <material name="black" />
+      </visual>
+      <inertial>
+        <origin xyz="0 0 0" rpy="${PI/2} 0 0" />
+        <mass value="${wheel_mass}" />
         <inertia
           ixx="${wheel_mass / 12.0 * (3*wheel_radius + wheel_len*wheel_len)}" ixy="0.0" ixz="0.0"
           iyy="${wheel_mass / 12.0 * wheel_radius*wheel_radius}" iyz="0.0"
-          izz="${wheel_mass / 12.0 * wheel_radius*wheel_radius}"/>
+          izz="${wheel_mass / 12.0 * wheel_radius*wheel_radius}" />
       </inertial>
     </link>
     <joint name="${prefix}caster_wheel_joint" type="fixed">
-      <parent link="${prefix}base_link"/>
-      <child link="${prefix}caster_wheel"/>
-      <origin xyz="${-base_length/2} 0 ${z_offset}" rpy="0 0 0"/> <!-- Updated caster wheel position -->
+      <parent link="${prefix}base_link" />
+      <child link="${prefix}caster_wheel" />
+      <origin xyz="${-base_length/2} 0 ${z_offset}" rpy="0 0 0" /> <!-- Updated caster wheel position -->
     </joint>
     <!-- caster wheel Link -->
     <link name="${prefix}caster_wheel">
       <collision>
-        <origin xyz="0 0 0" rpy="0 0 0"/>
-        <geometry>
-          <sphere radius="${caster_wheel_radius}"/>
-        </geometry>
-      </collision>
-      <visual>
-        <origin xyz="0 0 0" rpy="0 0 0"/>
-        <geometry>
-          <sphere radius="${caster_wheel_radius}"/>
-        </geometry>
-        <material name="white"/>
-      </visual>
-      <inertial>
-        <origin xyz="0 0 0" rpy="0 0 0"/>
-        <mass value="${caster_wheel_mass}"/>
-        <inertia
-              ixx="${2.0/5.0 * caster_wheel_mass * caster_wheel_radius * caster_wheel_radius}"
-              ixy="0.0" ixz="0.0"
-              iyy="${2.0/5.0 * caster_wheel_mass * caster_wheel_radius * caster_wheel_radius}"
-              iyz="0.0"
-              izz="${2.0/5.0 * caster_wheel_mass * caster_wheel_radius * caster_wheel_radius}"/>
-      </inertial>
-      </link>
-      <!-- laser_link -->
-      <link name="${prefix}laser_link">
-        <collision>
-          <origin xyz="${base_length/2} 0 ${base_height}" rpy="0 0 0"/>
-          <geometry>
-            <box size="0.1 0.1 0.1"/>
-          </geometry>
-        </collision>
-        <visual>
-          <origin xyz="${base_length/2} 0 ${base_height}" rpy="0 0 0"/>
-          <geometry>
-            <box size="0.1 0.1 0.1"/>
-          </geometry>
-          <material name="green"/>
-        </visual>
-        <inertial>
-          <origin xyz="${base_length/2} 0 ${base_height}" rpy="0 0 0"/>
-          <mass value="0.1"/>
-          <inertia
-            ixx="0.001" ixy="0.0" ixz="0.0"
-            iyy="0.001" iyz="0.0"
-            izz="0.001"/>
-        </inertial>
-      </link>
-      <!-- camera_link -->
-      <link name="${prefix}camera_link">
-        <collision>
-          <origin xyz="${base_length/2} 0 0" rpy="0 0 0"/>
-          <geometry>
-            <box size="0.1 0.1 0.1"/>
-          </geometry>
-        </collision>
-        <visual>
-          <origin xyz="${base_length/2} 0 0" rpy="0 0 0"/>
-          <geometry>
-            <box size="0.1 0.1 0.1"/>
-          </geometry>
-          <material name="blue"/>
-        </visual>
-        <inertial>
-          <origin xyz="${base_length/2} 0 0" rpy="0 0 0"/>
-          <mass value="0.1"/>
-          <inertia
-            ixx="0.001" ixy="0.0" ixz="0.0"
-            iyy="0.001" iyz="0.0"
-            izz="0.001"/>
-        </inertial>
-      </link>
-      <!-- Base Joint -->
-      <joint name="${prefix}base_joint" type="fixed">
-        <parent link="${prefix}base_link"/>
-        <child link="${prefix}laser_link"/>
-        <origin xyz="0 0 ${base_height}" rpy="0 0 0"/>
-      </joint>
-      <!-- Front Joint -->
-      <joint name="${prefix}front_joint" type="fixed">
-        <parent link="${prefix}laser_link"/>
-        <child link="${prefix}camera_link"/>
-        <origin xyz="${base_length/2} 0 ${base_height}" rpy="0 0 0"/>
-      </joint>
+        <origin xyz="0 0 0" rpy="0 0 0" />
+        <geometry>
+          <sphere radius="${caster_wheel_radius}" />
+        </geometry>
+      </collision>
+      <visual>
+        <origin xyz="0 0 0" rpy="0 0 0" />
+        <geometry>
+          <sphere radius="${caster_wheel_radius}" />
+        </geometry>
+        <material name="white" />
+      </visual>
+      <inertial>
+        <origin xyz="0 0 0" rpy="0 0 0" />
+        <mass value="${caster_wheel_mass}" />
+        <inertia
+          ixx="${2.0/5.0 * caster_wheel_mass * caster_wheel_radius * caster_wheel_radius}"
+          ixy="0.0" ixz="0.0"
+          iyy="${2.0/5.0 * caster_wheel_mass * caster_wheel_radius * caster_wheel_radius}"
+          iyz="0.0"
+          izz="${2.0/5.0 * caster_wheel_mass * caster_wheel_radius * caster_wheel_radius}" />
+      </inertial>
+    </link>
+    <!-- laser_link -->
+    <link name="${prefix}laser_link">
+      <collision>
+        <origin xyz="${base_length/2} 0 ${base_height}" rpy="0 0 0" />
+        <geometry>
+          <box size="0.1 0.1 0.1" />
+        </geometry>
+      </collision>
+      <visual>
+        <origin xyz="${base_length/2} 0 ${base_height}" rpy="0 0 0" />
+        <geometry>
+          <box size="0.1 0.1 0.1" />
+        </geometry>
+        <material name="green" />
+      </visual>
+      <inertial>
+        <origin xyz="${base_length/2} 0 ${base_height}" rpy="0 0 0" />
+        <mass value="0.1" />
+        <inertia
+          ixx="0.001" ixy="0.0" ixz="0.0"
+          iyy="0.001" iyz="0.0"
+          izz="0.001" />
+      </inertial>
+    </link>
+    <!-- camera_link -->
+    <link name="${prefix}camera_link">
+      <collision>
+        <origin xyz="${base_length/2} 0 0" rpy="0 0 0" />
+        <geometry>
+          <box size="0.1 0.1 0.1" />
+        </geometry>
+      </collision>
+      <visual>
+        <origin xyz="${base_length/2} 0 0" rpy="0 0 0" />
+        <geometry>
+          <box size="0.1 0.1 0.1" />
+        </geometry>
+        <material name="blue" />
+      </visual>
+      <inertial>
+        <origin xyz="${base_length/2} 0 0" rpy="0 0 0" />
+        <mass value="0.1" />
+        <inertia
+          ixx="0.001" ixy="0.0" ixz="0.0"
+          iyy="0.001" iyz="0.0"
+          izz="0.001" />
+      </inertial>
+    </link>
+    <!-- Base Joint -->
+    <joint name="${prefix}base_joint" type="fixed">
+      <parent link="${prefix}base_link" />
+      <child link="${prefix}laser_link" />
+      <origin xyz="0 0 ${base_height}" rpy="0 0 0" />
+    </joint>
+    <!-- Front Joint -->
+    <joint name="${prefix}front_joint" type="fixed">
+      <parent link="${prefix}laser_link" />
+      <child link="${prefix}camera_link" />
+      <origin xyz="${base_length/2} 0 ${base_height}" rpy="0 0 0" />
+    </joint>
   </xacro:macro>
 </robot>

File: urdf/odrive.urdf.xacro (robot description, xacro)
@@ -8,7 +8,7 @@
     <link name="link0" />
     <joint name="joint0" type="continuous">
-      <parent link="world"/>
-      <child link="link0"/>
-      <axis xyz="0 0 1"/>
+      <parent link="world" />
+      <child link="link0" />
+      <axis xyz="0 0 1" />
     </joint>
   </xacro:if>
@@ -16,7 +16,7 @@
     <link name="link1" />
     <joint name="joint1" type="continuous">
-      <parent link="world"/>
-      <child link="link1"/>
-      <axis xyz="0 0 1"/>
+      <parent link="world" />
+      <child link="link1" />
+      <axis xyz="0 0 1" />
     </joint>
   </xacro:if>

Commit message: update

File: urdf/diffbot.materials.xacro (robot description, xacro)
@@ -29,3 +29,9 @@
     <color rgba="1.0 1.0 1.0 1.0" />
   </material>
+  <material name="grey2">
+        <color rgba="0.9 0.9 0.9 1.0"/>
+  </material>
+  <material name="lightGrey">
+      <color rgba="0.6 0.6 0.6 1.0"/>
+  </material>
 </robot>

File: urdf/diffbot_description.urdf.xacro (robot description, xacro)
@@ -22,5 +22,5 @@
     <xacro:property name="chassis_offset" value="0.065"/>
     <!-- Materials -->
-    <material name="white">
+    <!-- <material name="white">
         <color rgba="1 1 1 1" />
     </material>
@@ -48,5 +48,5 @@
     <material name="lightGrey">
         <color rgba="0.6 0.6 0.6 1.0"/>
-    </material>
+    </material> -->
     <!-- Base Link -->
     <link name="${prefix}base_link">
