Commit message: update: fixes

File: urdf/diffbot_description.urdf.xacro (robot description, xacro)
@@ -32,5 +32,5 @@
             <origin xyz="1.2116163827517698533e-16 -0.47900000000000020339 -0.044999999999999998335" rpy="-5.5511151231257814695e-17 -0 3.141592653589793116" />
             <geometry>
-                <mesh filename="package:///right_motor.stl"/>
+                <mesh filename="file://$(find bot_mini_description)/mesh/right_motor.stl"/>
             </geometry>
             <material name="right_motor_material">
@@ -41,5 +41,5 @@
             <origin xyz="1.2116163827517698533e-16 -0.47900000000000020339 -0.044999999999999998335" rpy="-5.5511151231257814695e-17 -0 3.141592653589793116" />
             <geometry>
-                <mesh filename="package:///right_motor.stl"/>
+                <mesh filename="file://$(find bot_mini_description)/mesh/right_motor.stl"/>
             </geometry>
         </collision>
@@ -47,5 +47,5 @@
             <origin xyz="1.142227443712697323e-16 -0.47900000000000020339 -0.044999999999999998335" rpy="-5.5511151231257814695e-17 -0 3.141592653589793116" />
             <geometry>
-                <mesh filename="package:///motor_bar_frame.stl"/>
+                <mesh filename="file://$(find bot_mini_description)/mesh/motor_bar_frame.stl"/>
             </geometry>
             <material name="motor_bar_frame_material">
@@ -56,5 +56,5 @@
             <origin xyz="1.142227443712697323e-16 -0.47900000000000020339 -0.044999999999999998335" rpy="-5.5511151231257814695e-17 -0 3.141592653589793116" />
             <geometry>
-                <mesh filename="package:///motor_bar_frame.stl"/>
+                <mesh filename="file://$(find bot_mini_description)/mesh/motor_bar_frame.stl"/>
             </geometry>
         </collision>
@@ -62,5 +62,5 @@
             <origin xyz="1.142227443712697323e-16 -0.47900000000000020339 -0.044999999999999998335" rpy="-5.5511151231257814695e-17 -0 3.141592653589793116" />
             <geometry>
-                <mesh filename="package:///base_frame.stl"/>
+                <mesh filename="file://$(find bot_mini_description)/mesh/base_frame.stl"/>
             </geometry>
             <material name="base_frame_material">
@@ -71,5 +71,5 @@
             <origin xyz="1.142227443712697323e-16 -0.47900000000000020339 -0.044999999999999998335" rpy="-5.5511151231257814695e-17 -0 3.141592653589793116" />
             <geometry>
-                <mesh filename="package:///base_frame.stl"/>
+                <mesh filename="file://$(find bot_mini_description)/mesh/base_frame.stl"/>
             </geometry>
         </collision>
@@ -77,5 +77,5 @@
             <origin xyz="7.952827485173360274e-17 -0.4790000000000002589 -0.045000000000000012212" rpy="-5.5511151231257814695e-17 -0 3.141592653589793116" />
             <geometry>
-                <mesh filename="package:///left_motor.stl"/>
+                <mesh filename="file://$(find bot_mini_description)/mesh/left_motor.stl"/>
             </geometry>
             <material name="left_motor_material">
@@ -86,5 +86,5 @@
             <origin xyz="7.952827485173360274e-17 -0.4790000000000002589 -0.045000000000000012212" rpy="-5.5511151231257814695e-17 -0 3.141592653589793116" />
             <geometry>
-                <mesh filename="package:///left_motor.stl"/>
+                <mesh filename="file://$(find bot_mini_description)/mesh/left_motor.stl"/>
             </geometry>
         </collision>
@@ -92,5 +92,5 @@
             <origin xyz="7.4868290514223760072e-17 -0.47900000000000020339 -0.044999999999999998335" rpy="-5.5511151231257814695e-17 -0 3.141592653589793116" />
             <geometry>
-                <mesh filename="package:///caster_connector.stl"/>
+                <mesh filename="file://$(find bot_mini_description)/mesh/caster_connector.stl"/>
             </geometry>
             <material name="caster_connector_material">
@@ -101,5 +101,5 @@
             <origin xyz="7.4868290514223760072e-17 -0.47900000000000020339 -0.044999999999999998335" rpy="-5.5511151231257814695e-17 -0 3.141592653589793116" />
             <geometry>
-                <mesh filename="package:///caster_connector.stl"/>
+                <mesh filename="file://$(find bot_mini_description)/mesh/caster_connector.stl"/>
             </geometry>
         </collision>
@@ -107,5 +107,5 @@
             <origin xyz="1.1422274437126975695e-16 -0.47900000000000020339 -0.044999999999999998335" rpy="-5.5511151231257814695e-17 -0 3.141592653589793116" />
             <geometry>
-                <mesh filename="package:///right_motor_frame.stl"/>
+                <mesh filename="file://$(find bot_mini_description)/mesh/right_motor_frame.stl"/>
             </geometry>
             <material name="right_motor_frame_material">
@@ -116,5 +116,5 @@
             <origin xyz="1.1422274437126975695e-16 -0.47900000000000020339 -0.044999999999999998335" rpy="-5.5511151231257814695e-17 -0 3.141592653589793116" />
             <geometry>
-                <mesh filename="package:///right_motor_frame.stl"/>
+                <mesh filename="file://$(find bot_mini_description)/mesh/right_motor_frame.stl"/>
             </geometry>
         </collision>
@@ -122,5 +122,5 @@
             <origin xyz="8.6467168755640818792e-17 -0.47900000000000020339 -0.04500000000000002609" rpy="-5.5511151231257814695e-17 -0 3.141592653589793116" />
             <geometry>
-                <mesh filename="package:///left_motor_frame.stl"/>
+                <mesh filename="file://$(find bot_mini_description)/mesh/left_motor_frame.stl"/>
             </geometry>
             <material name="left_motor_frame_material">
@@ -131,5 +131,5 @@
             <origin xyz="8.6467168755640818792e-17 -0.47900000000000020339 -0.04500000000000002609" rpy="-5.5511151231257814695e-17 -0 3.141592653589793116" />
             <geometry>
-                <mesh filename="package:///left_motor_frame.stl"/>
+                <mesh filename="file://$(find bot_mini_description)/mesh/left_motor_frame.stl"/>
             </geometry>
         </collision>
@@ -137,5 +137,5 @@
             <origin xyz="7.4868290514223760072e-17 -0.47900000000000020339 -0.044999999999999998335" rpy="-5.5511151231257814695e-17 -0 3.141592653589793116" />
             <geometry>
-                <mesh filename="package:///caster_angle.stl"/>
+                <mesh filename="file://$(find bot_mini_description)/mesh/caster_angle.stl"/>
             </geometry>
             <material name="caster_angle_material">
@@ -146,5 +146,5 @@
             <origin xyz="7.4868290514223760072e-17 -0.47900000000000020339 -0.044999999999999998335" rpy="-5.5511151231257814695e-17 -0 3.141592653589793116" />
             <geometry>
-                <mesh filename="package:///caster_angle.stl"/>
+                <mesh filename="file://$(find bot_mini_description)/mesh/caster_angle.stl"/>
             </geometry>
         </collision>
@@ -169,5 +169,5 @@
             <origin xyz="-0.10999999999999998668 0.060000000000000011657 0.125" rpy="-1.570796326794896558 -1.570796326794896558 0" />
             <geometry>
-                <mesh filename="package:///left_wheel.stl"/>
+                <mesh filename="file://$(find bot_mini_description)/mesh/left_wheel.stl"/>
             </geometry>
             <material name="left_wheel_material">
@@ -178,5 +178,5 @@
             <origin xyz="-0.10999999999999998668 0.060000000000000011657 0.125" rpy="-1.570796326794896558 -1.570796326794896558 0" />
             <geometry>
-                <mesh filename="package:///left_wheel.stl"/>
+                <mesh filename="file://$(find bot_mini_description)/mesh/left_wheel.stl"/>
             </geometry>
         </collision>
@@ -201,5 +201,5 @@
             <origin xyz="-0.10999999999999998668 0.05999999999999999778 0.125" rpy="-1.570796326794896558 -1.570796326794896558 0" />
             <geometry>
-                <mesh filename="package:///left_wheel.stl"/>
+                <mesh filename="file://$(find bot_mini_description)/mesh/left_wheel.stl"/>
             </geometry>
             <material name="left_wheel_material">
@@ -210,5 +210,5 @@
             <origin xyz="-0.10999999999999998668 0.05999999999999999778 0.125" rpy="-1.570796326794896558 -1.570796326794896558 0" />
             <geometry>
-                <mesh filename="package:///left_wheel.stl"/>
+                <mesh filename="file://$(find bot_mini_description)/mesh/left_wheel.stl"/>
             </geometry>
         </collision>
@@ -233,5 +233,5 @@
             <origin xyz="1.1302212892091925974e-17 5.5511151231257827021e-17 0" rpy="3.141592653589793116 -8.3802055560433424155e-17 -3.141592653589793116" />
             <geometry>
-                <mesh filename="package:///caster_wheel.stl"/>
+                <mesh filename="file://$(find bot_mini_description)/mesh/caster_wheel.stl"/>
             </geometry>
             <material name="caster_wheel_material">
@@ -242,5 +242,5 @@
             <origin xyz="1.1302212892091925974e-17 5.5511151231257827021e-17 0" rpy="3.141592653589793116 -8.3802055560433424155e-17 -3.141592653589793116" />
             <geometry>
-                <mesh filename="package:///caster_wheel.stl"/>
+                <mesh filename="file://$(find bot_mini_description)/mesh/caster_wheel.stl"/>
             </geometry>
         </collision>
@@ -248,5 +248,5 @@
             <origin xyz="2.6961896103443574151e-18 0 0" rpy="3.141592653589793116 -0 0" />
             <geometry>
-                <mesh filename="package:///caster_bearing_frame.stl"/>
+                <mesh filename="file://$(find bot_mini_description)/mesh/caster_bearing_frame.stl"/>
             </geometry>
             <material name="caster_bearing_frame_material">
@@ -257,11 +257,11 @@
             <origin xyz="2.6961896103443574151e-18 0 0" rpy="3.141592653589793116 -0 0" />
             <geometry>
-                <mesh filename="package:///caster_bearing_frame.stl"/>
-            </geometry>
-        </collision>
-        <visual>
-            <origin xyz="-1.232595164407830946e-32 0 0" rpy="3.141592653589793116 4.7934256393637874986e-32 -3.141592653589793116" />
-            <geometry>
-                <mesh filename="package:///caster_frame_left.stl"/>
+                <mesh filename="file://$(find bot_mini_description)/mesh/caster_bearing_frame.stl"/>
+            </geometry>
+        </collision>
+        <visual>
+            <origin xyz="-1.232595164407830946e-32 0 0" rpy="3.141592653589793116 4.7934256393637874986e-32 -3.141592653589793116" />
+            <geometry>
+                <mesh filename="file://$(find bot_mini_description)/mesh/caster_frame_left.stl"/>
             </geometry>
             <material name="caster_frame_left_material">
@@ -272,11 +272,11 @@
             <origin xyz="-1.232595164407830946e-32 0 0" rpy="3.141592653589793116 4.7934256393637874986e-32 -3.141592653589793116" />
             <geometry>
-                <mesh filename="package:///caster_frame_left.stl"/>
-            </geometry>
-        </collision>
-        <visual>
-            <origin xyz="-1.232595164407830946e-32 0 0" rpy="3.141592653589793116 4.7934256393637874986e-32 -3.141592653589793116" />
-            <geometry>
-                <mesh filename="package:///caster_frame_top.stl"/>
+                <mesh filename="file://$(find bot_mini_description)/mesh/caster_frame_left.stl"/>
+            </geometry>
+        </collision>
+        <visual>
+            <origin xyz="-1.232595164407830946e-32 0 0" rpy="3.141592653589793116 4.7934256393637874986e-32 -3.141592653589793116" />
+            <geometry>
+                <mesh filename="file://$(find bot_mini_description)/mesh/caster_frame_top.stl"/>
             </geometry>
             <material name="caster_frame_top_material">
@@ -287,11 +287,11 @@
             <origin xyz="-1.232595164407830946e-32 0 0" rpy="3.141592653589793116 4.7934256393637874986e-32 -3.141592653589793116" />
             <geometry>
-                <mesh filename="package:///caster_frame_top.stl"/>
-            </geometry>
-        </collision>
-        <visual>
-            <origin xyz="-1.232595164407830946e-32 0 0" rpy="3.141592653589793116 4.7934256393637874986e-32 -3.141592653589793116" />
-            <geometry>
-                <mesh filename="package:///caster_frame_right.stl"/>
+                <mesh filename="file://$(find bot_mini_description)/mesh/caster_frame_top.stl"/>
+            </geometry>
+        </collision>
+        <visual>
+            <origin xyz="-1.232595164407830946e-32 0 0" rpy="3.141592653589793116 4.7934256393637874986e-32 -3.141592653589793116" />
+            <geometry>
+                <mesh filename="file://$(find bot_mini_description)/mesh/caster_frame_right.stl"/>
             </geometry>
             <material name="caster_frame_right_material">
@@ -302,5 +302,5 @@
             <origin xyz="-1.232595164407830946e-32 0 0" rpy="3.141592653589793116 4.7934256393637874986e-32 -3.141592653589793116" />
             <geometry>
-                <mesh filename="package:///caster_frame_right.stl"/>
+                <mesh filename="file://$(find bot_mini_description)/mesh/caster_frame_right.stl"/>
             </geometry>
         </collision>
@@ -316,5 +316,5 @@
             <origin xyz="-4.1223423760908350982e-18 0.13500000000000000888 0.025000000000000001388" rpy="3.141592653589793116 -0 1.0263416486754026723e-48" />
             <geometry>
-                <mesh filename="package:///laser_frame.stl"/>
+                <mesh filename="file://$(find bot_mini_description)/mesh/laser_frame.stl"/>
             </geometry>
             <material name="laser_frame_material">
@@ -325,5 +325,5 @@
             <origin xyz="-4.1223423760908350982e-18 0.13500000000000000888 0.025000000000000001388" rpy="3.141592653589793116 -0 1.0263416486754026723e-48" />
             <geometry>
-                <mesh filename="package:///laser_frame.stl"/>
+                <mesh filename="file://$(find bot_mini_description)/mesh/laser_frame.stl"/>
             </geometry>
         </collision>
@@ -348,5 +348,5 @@
             <origin xyz="3.0814879110195773649e-32 0 0" rpy="-1.570796326794896558 2.775557561562890365e-16 -9.2444637330585569324e-33" />
             <geometry>
-                <mesh filename="package:///camera_frame.stl"/>
+                <mesh filename="file://$(find bot_mini_description)/mesh/camera_frame.stl"/>
             </geometry>
             <material name="hikvision_ds-u02_material">
@@ -357,5 +357,5 @@
             <origin xyz="3.0814879110195773649e-32 0 0" rpy="-1.570796326794896558 2.775557561562890365e-16 -9.2444637330585569324e-33" />
             <geometry>
-                <mesh filename="package:///camera_frame.stl"/>
+                <mesh filename="file://$(find bot_mini_description)/mesh/camera_frame.stl"/>
             </geometry>
         </collision>

Commit message: update: continuous joints

File: urdf/diffbot_description.urdf.xacro (robot description, xacro)
@@ -156,5 +156,5 @@
     </link>
     <!-- right wheel joint -->
-    <joint name="${prefix}right_wheel_joint" type="revolute">
+    <joint name="${prefix}right_wheel_joint" type="continuous">
       <origin xyz="-0.12499999999999993061 -0.58900000000000007905 -0.10500000000000000999" rpy="-1.570796326794896558 -2.2204460492503130808e-16 -1.57079632679489678" />
 <parent link="${prefix}base_link" />
@@ -188,5 +188,5 @@
     </link>
     <!-- left wheel joint -->
-    <joint name="${prefix}left_wheel_joint" type="revolute">
+    <joint name="${prefix}left_wheel_joint" type="continuous">
       <origin xyz="0.12500000000000013878 -0.58900000000000007905 -0.10500000000000003775" rpy="1.57079632679489678 -1.1102230246251567869e-16 -1.570796326794896558" />
       <parent link="${prefix}base_link" />
@@ -220,5 +220,5 @@
     </link>
     <!-- caster wheel joint -->
-    <joint name="${prefix}caster_wheel_joint" type="revolute">
+    <joint name="${prefix}caster_wheel_joint" type="continuous">
         <origin xyz="5.3368019332749957491e-17 -0.29900000000000009903 -0.064999999999999974465" rpy="-5.5511151231257814695e-17 -0 3.141592653589793116" />
         <parent link="${prefix}base_link" />
@@ -335,5 +335,5 @@
     </link>
     <!-- laser_joint -->
-    <joint name="${prefix}laser_joint" type="revolute">
+    <joint name="${prefix}laser_joint" type="continuous">
         <origin xyz="8.9609515272227915335e-17 -0.61400000000000021227 -0.019999999999999972661" rpy="-3.141592653589793116 -6.1629758220391519929e-33 1.1102230246251560474e-16" />
         <parent link="${prefix}base_link" />
@@ -367,5 +367,5 @@
     </link>
     <!-- Camera Joint -->
-    <joint name="${prefix}camera_joint" type="revolute">
+    <joint name="${prefix}camera_joint" type="continuous">
         <origin xyz="9.7569399001892381731e-17 -0.6290000000000002256 -0.045000000000000005274" rpy="6.1062266354383530837e-16 1.1102230246251567869e-16 3.141592653589793116" />
         <parent link="${prefix}base_link" />
