Commit message: update

File: urdf/diffbot_description.urdf.xacro (robot description, xacro)
@@ -29,161 +29,161 @@
     <!-- Base Link -->
     <link name="${prefix}base_link">
-        <visual>
-            <origin xyz="1.2116163827517698533e-16 -0.47900000000000020339 -0.044999999999999998335" rpy="-5.5511151231257814695e-17 -0 3.141592653589793116" />
-            <geometry>
-                <mesh filename="file://$(find bot_mini_description)/mesh/right_motor.stl"/>
-            </geometry>
-            <material name="right_motor_material">
-                <color rgba="0.49803921568627451677 0.49803921568627451677 0.49803921568627451677 1.0"/>
-            </material>
-        </visual>
-        <collision>
-            <origin xyz="1.2116163827517698533e-16 -0.47900000000000020339 -0.044999999999999998335" rpy="-5.5511151231257814695e-17 -0 3.141592653589793116" />
-            <geometry>
-                <mesh filename="file://$(find bot_mini_description)/mesh/right_motor.stl"/>
-            </geometry>
-        </collision>
-        <visual>
-            <origin xyz="1.142227443712697323e-16 -0.47900000000000020339 -0.044999999999999998335" rpy="-5.5511151231257814695e-17 -0 3.141592653589793116" />
-            <geometry>
-                <mesh filename="file://$(find bot_mini_description)/mesh/motor_bar_frame.stl"/>
-            </geometry>
-            <material name="motor_bar_frame_material">
-                <color rgba="0.91764705882352937127 0.91764705882352937127 0.91764705882352937127 1.0"/>
-            </material>
-        </visual>
-        <collision>
-            <origin xyz="1.142227443712697323e-16 -0.47900000000000020339 -0.044999999999999998335" rpy="-5.5511151231257814695e-17 -0 3.141592653589793116" />
-            <geometry>
-                <mesh filename="file://$(find bot_mini_description)/mesh/motor_bar_frame.stl"/>
-            </geometry>
-        </collision>
-        <visual>
-            <origin xyz="1.142227443712697323e-16 -0.47900000000000020339 -0.044999999999999998335" rpy="-5.5511151231257814695e-17 -0 3.141592653589793116" />
-            <geometry>
-                <mesh filename="file://$(find bot_mini_description)/mesh/base_frame.stl"/>
-            </geometry>
-            <material name="base_frame_material">
-                <color rgba="0.91764705882352937127 0.91764705882352937127 0.91764705882352937127 1.0"/>
-            </material>
-        </visual>
-        <collision>
-            <origin xyz="1.142227443712697323e-16 -0.47900000000000020339 -0.044999999999999998335" rpy="-5.5511151231257814695e-17 -0 3.141592653589793116" />
-            <geometry>
-                <mesh filename="file://$(find bot_mini_description)/mesh/base_frame.stl"/>
-            </geometry>
-        </collision>
-        <visual>
-            <origin xyz="7.952827485173360274e-17 -0.4790000000000002589 -0.045000000000000012212" rpy="-5.5511151231257814695e-17 -0 3.141592653589793116" />
-            <geometry>
-                <mesh filename="file://$(find bot_mini_description)/mesh/left_motor.stl"/>
-            </geometry>
-            <material name="left_motor_material">
-                <color rgba="0.49803921568627451677 0.49803921568627451677 0.49803921568627451677 1.0"/>
-            </material>
-        </visual>
-        <collision>
-            <origin xyz="7.952827485173360274e-17 -0.4790000000000002589 -0.045000000000000012212" rpy="-5.5511151231257814695e-17 -0 3.141592653589793116" />
-            <geometry>
-                <mesh filename="file://$(find bot_mini_description)/mesh/left_motor.stl"/>
-            </geometry>
-        </collision>
-        <visual>
-            <origin xyz="7.4868290514223760072e-17 -0.47900000000000020339 -0.044999999999999998335" rpy="-5.5511151231257814695e-17 -0 3.141592653589793116" />
-            <geometry>
-                <mesh filename="file://$(find bot_mini_description)/mesh/caster_connector.stl"/>
-            </geometry>
-            <material name="caster_connector_material">
-                <color rgba="0.91764705882352937127 0.91764705882352937127 0.91764705882352937127 1.0"/>
-            </material>
-        </visual>
-        <collision>
-            <origin xyz="7.4868290514223760072e-17 -0.47900000000000020339 -0.044999999999999998335" rpy="-5.5511151231257814695e-17 -0 3.141592653589793116" />
-            <geometry>
-                <mesh filename="file://$(find bot_mini_description)/mesh/caster_connector.stl"/>
-            </geometry>
-        </collision>
-        <visual>
-            <origin xyz="1.1422274437126975695e-16 -0.47900000000000020339 -0.044999999999999998335" rpy="-5.5511151231257814695e-17 -0 3.141592653589793116" />
-            <geometry>
-                <mesh filename="file://$(find bot_mini_description)/mesh/right_motor_frame.stl"/>
-            </geometry>
-            <material name="right_motor_frame_material">
-                <color rgba="0.08627450980392156743 0.31764705882352939348 0.69019607843137253944 1.0"/>
-            </material>
-        </visual>
-        <collision>
-            <origin xyz="1.1422274437126975695e-16 -0.47900000000000020339 -0.044999999999999998335" rpy="-5.5511151231257814695e-17 -0 3.141592653589793116" />
-            <geometry>
-                <mesh filename="file://$(find bot_mini_description)/mesh/right_motor_frame.stl"/>
-            </geometry>
-        </collision>
-        <visual>
-            <origin xyz="8.6467168755640818792e-17 -0.47900000000000020339 -0.04500000000000002609" rpy="-5.5511151231257814695e-17 -0 3.141592653589793116" />
-            <geometry>
-                <mesh filename="file://$(find bot_mini_description)/mesh/left_motor_frame.stl"/>
-            </geometry>
-            <material name="left_motor_frame_material">
-                <color rgba="0.08627450980392156743 0.31764705882352939348 0.69019607843137253944 1.0"/>
-            </material>
-        </visual>
-        <collision>
-            <origin xyz="8.6467168755640818792e-17 -0.47900000000000020339 -0.04500000000000002609" rpy="-5.5511151231257814695e-17 -0 3.141592653589793116" />
-            <geometry>
-                <mesh filename="file://$(find bot_mini_description)/mesh/left_motor_frame.stl"/>
-            </geometry>
-        </collision>
-        <visual>
-            <origin xyz="7.4868290514223760072e-17 -0.47900000000000020339 -0.044999999999999998335" rpy="-5.5511151231257814695e-17 -0 3.141592653589793116" />
-            <geometry>
-                <mesh filename="file://$(find bot_mini_description)/mesh/caster_angle.stl"/>
-            </geometry>
-            <material name="caster_angle_material">
-                <color rgba="0.64705882352941179736 0.64705882352941179736 0.64705882352941179736 1.0"/>
-            </material>
-        </visual>
-        <collision>
-            <origin xyz="7.4868290514223760072e-17 -0.47900000000000020339 -0.044999999999999998335" rpy="-5.5511151231257814695e-17 -0 3.141592653589793116" />
-            <geometry>
-                <mesh filename="file://$(find bot_mini_description)/mesh/caster_angle.stl"/>
-            </geometry>
-        </collision>
-        <inertial>
-            <origin xyz="7.8969938888060694711e-17 -0.50510328199237819469 -0.048726182398186372591" rpy="0 0 0"/>
-            <mass value="8.4123950268139715547" />
-            <inertia ixx="0.090166990291185411532" ixy="1.2345824367636969194e-17" ixz="2.072268733803397153e-18" iyy="0.055481261106946754003" iyz="-0.011121590612260267433" izz="0.13051099377067154617" />
-        </inertial>
+      <visual>
+        <origin xyz="1.2116163827517698533e-16 -0.47900000000000020339 -0.044999999999999998335" rpy="-5.5511151231257814695e-17 -0 3.141592653589793116" />
+        <geometry>
+          <mesh filename="file://$(find bot_mini_description)/mesh/right_motor.stl"/>
+        </geometry>
+        <material name="right_motor_material">
+          <color rgba="0.49803921568627451677 0.49803921568627451677 0.49803921568627451677 1.0"/>
+        </material>
+      </visual>
+      <collision>
+        <origin xyz="1.2116163827517698533e-16 -0.47900000000000020339 -0.044999999999999998335" rpy="-5.5511151231257814695e-17 -0 3.141592653589793116" />
+        <geometry>
+          <mesh filename="file://$(find bot_mini_description)/mesh/right_motor.stl"/>
+        </geometry>
+      </collision>
+      <visual>
+        <origin xyz="1.142227443712697323e-16 -0.47900000000000020339 -0.044999999999999998335" rpy="-5.5511151231257814695e-17 -0 3.141592653589793116" />
+        <geometry>
+          <mesh filename="file://$(find bot_mini_description)/mesh/motor_bar_frame.stl"/>
+        </geometry>
+        <material name="motor_bar_frame_material">
+          <color rgba="0.91764705882352937127 0.91764705882352937127 0.91764705882352937127 1.0"/>
+        </material>
+      </visual>
+      <collision>
+        <origin xyz="1.142227443712697323e-16 -0.47900000000000020339 -0.044999999999999998335" rpy="-5.5511151231257814695e-17 -0 3.141592653589793116" />
+        <geometry>
+          <mesh filename="file://$(find bot_mini_description)/mesh/motor_bar_frame.stl"/>
+        </geometry>
+      </collision>
+      <visual>
+        <origin xyz="1.142227443712697323e-16 -0.47900000000000020339 -0.044999999999999998335" rpy="-5.5511151231257814695e-17 -0 3.141592653589793116" />
+        <geometry>
+          <mesh filename="file://$(find bot_mini_description)/mesh/base_frame.stl"/>
+        </geometry>
+        <material name="base_frame_material">
+          <color rgba="0.91764705882352937127 0.91764705882352937127 0.91764705882352937127 1.0"/>
+        </material>
+      </visual>
+      <collision>
+        <origin xyz="1.142227443712697323e-16 -0.47900000000000020339 -0.044999999999999998335" rpy="-5.5511151231257814695e-17 -0 3.141592653589793116" />
+        <geometry>
+          <mesh filename="file://$(find bot_mini_description)/mesh/base_frame.stl"/>
+        </geometry>
+      </collision>
+      <visual>
+        <origin xyz="7.952827485173360274e-17 -0.4790000000000002589 -0.045000000000000012212" rpy="-5.5511151231257814695e-17 -0 3.141592653589793116" />
+        <geometry>
+          <mesh filename="file://$(find bot_mini_description)/mesh/left_motor.stl"/>
+        </geometry>
+        <material name="left_motor_material">
+          <color rgba="0.49803921568627451677 0.49803921568627451677 0.49803921568627451677 1.0"/>
+        </material>
+      </visual>
+      <collision>
+        <origin xyz="7.952827485173360274e-17 -0.4790000000000002589 -0.045000000000000012212" rpy="-5.5511151231257814695e-17 -0 3.141592653589793116" />
+        <geometry>
+          <mesh filename="file://$(find bot_mini_description)/mesh/left_motor.stl"/>
+        </geometry>
+      </collision>
+      <visual>
+        <origin xyz="7.4868290514223760072e-17 -0.47900000000000020339 -0.044999999999999998335" rpy="-5.5511151231257814695e-17 -0 3.141592653589793116" />
+        <geometry>
+          <mesh filename="file://$(find bot_mini_description)/mesh/caster_connector.stl"/>
+        </geometry>
+        <material name="caster_connector_material">
+          <color rgba="0.91764705882352937127 0.91764705882352937127 0.91764705882352937127 1.0"/>
+        </material>
+      </visual>
+      <collision>
+        <origin xyz="7.4868290514223760072e-17 -0.47900000000000020339 -0.044999999999999998335" rpy="-5.5511151231257814695e-17 -0 3.141592653589793116" />
+        <geometry>
+          <mesh filename="file://$(find bot_mini_description)/mesh/caster_connector.stl"/>
+        </geometry>
+      </collision>
+      <visual>
+        <origin xyz="1.1422274437126975695e-16 -0.47900000000000020339 -0.044999999999999998335" rpy="-5.5511151231257814695e-17 -0 3.141592653589793116" />
+        <geometry>
+          <mesh filename="file://$(find bot_mini_description)/mesh/right_motor_frame.stl"/>
+        </geometry>
+        <material name="right_motor_frame_material">
+          <color rgba="0.08627450980392156743 0.31764705882352939348 0.69019607843137253944 1.0"/>
+        </material>
+      </visual>
+      <collision>
+        <origin xyz="1.1422274437126975695e-16 -0.47900000000000020339 -0.044999999999999998335" rpy="-5.5511151231257814695e-17 -0 3.141592653589793116" />
+        <geometry>
+          <mesh filename="file://$(find bot_mini_description)/mesh/right_motor_frame.stl"/>
+        </geometry>
+      </collision>
+      <visual>
+        <origin xyz="8.6467168755640818792e-17 -0.47900000000000020339 -0.04500000000000002609" rpy="-5.5511151231257814695e-17 -0 3.141592653589793116" />
+        <geometry>
+          <mesh filename="file://$(find bot_mini_description)/mesh/left_motor_frame.stl"/>
+        </geometry>
+        <material name="left_motor_frame_material">
+          <color rgba="0.08627450980392156743 0.31764705882352939348 0.69019607843137253944 1.0"/>
+        </material>
+      </visual>
+      <collision>
+        <origin xyz="8.6467168755640818792e-17 -0.47900000000000020339 -0.04500000000000002609" rpy="-5.5511151231257814695e-17 -0 3.141592653589793116" />
+        <geometry>
+          <mesh filename="file://$(find bot_mini_description)/mesh/left_motor_frame.stl"/>
+        </geometry>
+      </collision>
+      <visual>
+        <origin xyz="7.4868290514223760072e-17 -0.47900000000000020339 -0.044999999999999998335" rpy="-5.5511151231257814695e-17 -0 3.141592653589793116" />
+        <geometry>
+          <mesh filename="file://$(find bot_mini_description)/mesh/caster_angle.stl"/>
+        </geometry>
+        <material name="caster_angle_material">
+          <color rgba="0.64705882352941179736 0.64705882352941179736 0.64705882352941179736 1.0"/>
+        </material>
+      </visual>
+      <collision>
+        <origin xyz="7.4868290514223760072e-17 -0.47900000000000020339 -0.044999999999999998335" rpy="-5.5511151231257814695e-17 -0 3.141592653589793116" />
+        <geometry>
+          <mesh filename="file://$(find bot_mini_description)/mesh/caster_angle.stl"/>
+        </geometry>
+      </collision>
+      <inertial>
+        <origin xyz="7.8969938888060694711e-17 -0.50510328199237819469 -0.048726182398186372591" rpy="0 0 0"/>
+        <mass value="8.4123950268139715547" />
+        <inertia ixx="0.090166990291185411532" ixy="1.2345824367636969194e-17" ixz="2.072268733803397153e-18" iyy="0.055481261106946754003" iyz="-0.011121590612260267433" izz="0.13051099377067154617" />
+      </inertial>
     </link>
     <!-- right wheel joint -->
     <joint name="${prefix}right_wheel_joint" type="continuous">
       <origin xyz="-0.12499999999999993061 -0.58900000000000007905 -0.10500000000000000999" rpy="-1.570796326794896558 -2.2204460492503130808e-16 -1.57079632679489678" />
-<parent link="${prefix}base_link" />
-<child link="${prefix}right_wheel_link" />
-<axis xyz="0 0 1"/>
-<limit effort="1" velocity="20" />
-<joint_properties friction="0.0"/>
-</joint>
+      <parent link="${prefix}base_link" />
+      <child link="${prefix}right_wheel_link" />
+      <axis xyz="0 0 1"/>
+      <limit effort="1" velocity="20" />
+      <joint_properties friction="0.0"/>
+    </joint>
     <!-- right wheel Link -->
     <link name="${prefix}right_wheel_link">
-        <visual>
-            <origin xyz="-0.10999999999999998668 0.060000000000000011657 0.125" rpy="-1.570796326794896558 -1.570796326794896558 0" />
-            <geometry>
-                <mesh filename="file://$(find bot_mini_description)/mesh/left_wheel.stl"/>
-            </geometry>
-            <material name="left_wheel_material">
-                <color rgba="0.50196078431372548323 0.50196078431372548323 0.50196078431372548323 1.0"/>
-            </material>
-        </visual>
-        <collision>
-            <origin xyz="-0.10999999999999998668 0.060000000000000011657 0.125" rpy="-1.570796326794896558 -1.570796326794896558 0" />
-            <geometry>
-                <mesh filename="file://$(find bot_mini_description)/mesh/left_wheel.stl"/>
-            </geometry>
-        </collision>
-        <inertial>
-            <origin xyz="1.3877787807814456755e-17 1.3877787807814456755e-17 -0.017500000000000015543" rpy="0 0 0"/>
-            <mass value="0.43298678305638949038" />
-            <inertia ixx="0.00043196650576949035269" ixy="0" ixz="1.8666117243005040269e-36" iyy="0.00043196650576949029848" iyz="0" izz="0.00078373880522818965139" />
-        </inertial>
+      <visual>
+        <origin xyz="-0.10999999999999998668 0.060000000000000011657 0.125" rpy="-1.570796326794896558 -1.570796326794896558 0" />
+        <geometry>
+          <mesh filename="file://$(find bot_mini_description)/mesh/left_wheel.stl"/>
+        </geometry>
+        <material name="left_wheel_material">
+          <color rgba="0.50196078431372548323 0.50196078431372548323 0.50196078431372548323 1.0"/>
+        </material>
+      </visual>
+      <collision>
+        <origin xyz="-0.10999999999999998668 0.060000000000000011657 0.125" rpy="-1.570796326794896558 -1.570796326794896558 0" />
+        <geometry>
+          <mesh filename="file://$(find bot_mini_description)/mesh/left_wheel.stl"/>
+        </geometry>
+      </collision>
+      <inertial>
+        <origin xyz="1.3877787807814456755e-17 1.3877787807814456755e-17 -0.017500000000000015543" rpy="0 0 0"/>
+        <mass value="0.43298678305638949038" />
+        <inertia ixx="0.00043196650576949035269" ixy="0" ixz="1.8666117243005040269e-36" iyy="0.00043196650576949029848" iyz="0" izz="0.00078373880522818965139" />
+      </inertial>
     </link>
     <!-- left wheel joint -->
@@ -197,181 +197,181 @@
     </joint>
     <!-- left wheel Link -->
-    <link name="left_wheel_link">
-        <visual>
-            <origin xyz="-0.10999999999999998668 0.05999999999999999778 0.125" rpy="-1.570796326794896558 -1.570796326794896558 0" />
-            <geometry>
-                <mesh filename="file://$(find bot_mini_description)/mesh/left_wheel.stl"/>
-            </geometry>
-            <material name="left_wheel_material">
-                <color rgba="0.50196078431372548323 0.50196078431372548323 0.50196078431372548323 1.0"/>
-            </material>
-        </visual>
-        <collision>
-            <origin xyz="-0.10999999999999998668 0.05999999999999999778 0.125" rpy="-1.570796326794896558 -1.570796326794896558 0" />
-            <geometry>
-                <mesh filename="file://$(find bot_mini_description)/mesh/left_wheel.stl"/>
-            </geometry>
-        </collision>
-        <inertial>
-            <origin xyz="1.3877787807814456755e-17 0 -0.017500000000000015543" rpy="0 0 0"/>
-            <mass value="0.43298678305638949038" />
-            <inertia ixx="0.00043196650576949035269" ixy="1.4778173856800390343e-52" ixz="-4.8081924471597460774e-36" iyy="0.00043196650576949029848" iyz="0" izz="0.00078373880522818965139" />
-        </inertial>
+    <link name="${prefix}left_wheel_link">
+      <visual>
+        <origin xyz="-0.10999999999999998668 0.05999999999999999778 0.125" rpy="-1.570796326794896558 -1.570796326794896558 0" />
+        <geometry>
+          <mesh filename="file://$(find bot_mini_description)/mesh/left_wheel.stl"/>
+        </geometry>
+        <material name="left_wheel_material">
+          <color rgba="0.50196078431372548323 0.50196078431372548323 0.50196078431372548323 1.0"/>
+        </material>
+      </visual>
+      <collision>
+        <origin xyz="-0.10999999999999998668 0.05999999999999999778 0.125" rpy="-1.570796326794896558 -1.570796326794896558 0" />
+        <geometry>
+          <mesh filename="file://$(find bot_mini_description)/mesh/left_wheel.stl"/>
+        </geometry>
+      </collision>
+      <inertial>
+        <origin xyz="1.3877787807814456755e-17 0 -0.017500000000000015543" rpy="0 0 0"/>
+        <mass value="0.43298678305638949038" />
+        <inertia ixx="0.00043196650576949035269" ixy="1.4778173856800390343e-52" ixz="-4.8081924471597460774e-36" iyy="0.00043196650576949029848" iyz="0" izz="0.00078373880522818965139" />
+      </inertial>
     </link>
     <!-- caster wheel joint -->
     <joint name="${prefix}caster_wheel_joint" type="continuous">
-        <origin xyz="5.3368019332749957491e-17 -0.29900000000000009903 -0.064999999999999974465" rpy="-5.5511151231257814695e-17 -0 3.141592653589793116" />
-        <parent link="${prefix}base_link" />
-        <child link="${prefix}caster_wheel_link" />
-        <axis xyz="0 0 1"/>
-        <limit effort="1" velocity="20" />
-        <joint_properties friction="0.0"/>
+      <origin xyz="5.3368019332749957491e-17 -0.29900000000000009903 -0.064999999999999974465" rpy="-5.5511151231257814695e-17 -0 3.141592653589793116" />
+      <parent link="${prefix}base_link" />
+      <child link="${prefix}caster_wheel_link" />
+      <axis xyz="0 0 1"/>
+      <limit effort="1" velocity="20" />
+      <joint_properties friction="0.0"/>
     </joint>
     <!-- caster wheel Link -->
     <link name="${prefix}caster_wheel_link">
-        <visual>
-            <origin xyz="1.1302212892091925974e-17 5.5511151231257827021e-17 0" rpy="3.141592653589793116 -8.3802055560433424155e-17 -3.141592653589793116" />
-            <geometry>
-                <mesh filename="file://$(find bot_mini_description)/mesh/caster_wheel.stl"/>
-            </geometry>
-            <material name="caster_wheel_material">
-                <color rgba="0.50196078431372548323 0.50196078431372548323 0.50196078431372548323 1.0"/>
-            </material>
-        </visual>
-        <collision>
-            <origin xyz="1.1302212892091925974e-17 5.5511151231257827021e-17 0" rpy="3.141592653589793116 -8.3802055560433424155e-17 -3.141592653589793116" />
-            <geometry>
-                <mesh filename="file://$(find bot_mini_description)/mesh/caster_wheel.stl"/>
-            </geometry>
-        </collision>
-        <visual>
-            <origin xyz="2.6961896103443574151e-18 0 0" rpy="3.141592653589793116 -0 0" />
-            <geometry>
-                <mesh filename="file://$(find bot_mini_description)/mesh/caster_bearing_frame.stl"/>
-            </geometry>
-            <material name="caster_bearing_frame_material">
-                <color rgba="0.80000000000000004441 0.80000000000000004441 0.80000000000000004441 1.0"/>
-            </material>
-        </visual>
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
File: urdf/odrive.ros2_control.xacro (robot description, xacro)
@@ -22,5 +22,5 @@
           <param name="serial_number">${serial_number}</param>
           <param name="axis">1</param>
-          <param name="enable_watchdog">1</param>
+          <param name="enable_watchdog">0</param>
           <param name="watchdog_timeout">0.1</param>
         </joint>
