Commit message: fixes for slam toolbox

File: urdf/diffbot_description.urdf.xacro (robot description, xacro)
@@ -155,4 +155,25 @@
       </inertial>
     </link>
+    <!-- Adding base_footprint for mapping (Needed by slam toolbox) -->
+    <link name="${prefix}base_footprint">
+      <collision>
+        <origin xyz="0 0 0" rpy="0 0 0"/>
+        <geometry>
+          <box size="${base_length} ${base_width} ${base_height}"/> <!-- Updated base dimensions -->
+        </geometry>
+      </collision>
+      <visual>
+        <origin xyz="0 0 ${base_height/2}" rpy="0 0 0"/>
+        <geometry>
+          <box size="${base_length} ${base_width} ${base_height}"/> <!-- Updated base dimensions -->
+        </geometry>
+        <material name="orange"/>
+      </visual>
+    </link>
+    <joint name="${prefix}base_footprint_joint" type="fixed">
+      <origin xyz="0 0 0" rpy="0 0 0" />
+      <parent link="${prefix}base_link" />
+      <child link="${prefix}base_footprint" />
+    </joint>
     <!-- right wheel joint -->
     <joint name="${prefix}right_wheel_joint" type="continuous">

Commit message: update

File: urdf/diffbot_description.urdf.xacro (robot description, xacro)
@@ -172,5 +172,4 @@
     </link>
     <joint name="${prefix}base_footprint_joint" type="fixed">
-      <origin xyz="0 0 0" rpy="0 0 0" />
       <parent link="${prefix}base_link" />
       <child link="${prefix}base_footprint" />

Commit message: update: fixes

File: urdf/diffbot_description.urdf.xacro (robot description, xacro)
@@ -157,17 +157,4 @@
     <!-- Adding base_footprint for mapping (Needed by slam toolbox) -->
     <link name="${prefix}base_footprint">
-      <collision>
-        <origin xyz="0 0 0" rpy="0 0 0"/>
-        <geometry>
-          <box size="${base_length} ${base_width} ${base_height}"/> <!-- Updated base dimensions -->
-        </geometry>
-      </collision>
-      <visual>
-        <origin xyz="0 0 ${base_height/2}" rpy="0 0 0"/>
-        <geometry>
-          <box size="${base_length} ${base_width} ${base_height}"/> <!-- Updated base dimensions -->
-        </geometry>
-        <material name="orange"/>
-      </visual>
     </link>
     <joint name="${prefix}base_footprint_joint" type="fixed">
@@ -240,5 +227,5 @@
     </link>
     <!-- caster wheel joint -->
-    <joint name="${prefix}caster_wheel_joint" type="continuous">
+    <joint name="${prefix}caster_wheel_joint" type="fixed">
       <origin xyz="5.3368019332749957491e-17 -0.29900000000000009903 -0.064999999999999974465" rpy="-5.5511151231257814695e-17 -0 3.141592653589793116" />
       <parent link="${prefix}base_link" />
@@ -355,5 +342,5 @@
     </link>
     <!-- laser_joint -->
-    <joint name="${prefix}laser_joint" type="continuous">
+    <joint name="${prefix}laser_joint" type="fixed">
       <origin xyz="8.9609515272227915335e-17 -0.61400000000000021227 -0.019999999999999972661" rpy="-3.141592653589793116 -6.1629758220391519929e-33 1.1102230246251560474e-16" />
       <parent link="${prefix}base_link" />
@@ -387,5 +374,5 @@
     </link>
     <!-- Camera Joint -->
-    <joint name="${prefix}camera_joint" type="continuous">
+    <joint name="${prefix}camera_joint" type="fixed">
       <origin xyz="9.7569399001892381731e-17 -0.6290000000000002256 -0.045000000000000005274" rpy="6.1062266354383530837e-16 1.1102230246251567869e-16 3.141592653589793116" />
       <parent link="${prefix}base_link" />

Commit message: fixes for wheels

File: urdf/diffbot_description.urdf.xacro (robot description, xacro)
@@ -166,5 +166,5 @@
       <origin xyz="-0.12499999999999993061 -0.58900000000000007905 -0.10500000000000000999" rpy="-1.570796326794896558 -2.2204460492503130808e-16 -1.57079632679489678" />
       <parent link="${prefix}base_link" />
-      <child link="${prefix}right_wheel_link" />
+      <child link="${prefix}right_wheel" />
       <axis xyz="0 0 1"/>
       <limit effort="1" velocity="20" />
@@ -172,5 +172,5 @@
     </joint>
     <!-- right wheel Link -->
-    <link name="${prefix}right_wheel_link">
+    <link name="${prefix}right_wheel">
       <visual>
         <origin xyz="-0.10999999999999998668 0.060000000000000011657 0.125" rpy="-1.570796326794896558 -1.570796326794896558 0" />
@@ -198,5 +198,5 @@
       <origin xyz="0.12500000000000013878 -0.58900000000000007905 -0.10500000000000003775" rpy="1.57079632679489678 -1.1102230246251567869e-16 -1.570796326794896558" />
       <parent link="${prefix}base_link" />
-      <child link="${prefix}left_wheel_link" />
+      <child link="${prefix}left_wheel" />
       <axis xyz="0 0 1" />
       <limit effort="1" velocity="20" />
@@ -204,5 +204,5 @@
     </joint>
     <!-- left wheel Link -->
-    <link name="${prefix}left_wheel_link">
+    <link name="${prefix}left_wheel">
       <visual>
         <origin xyz="-0.10999999999999998668 0.05999999999999999778 0.125" rpy="-1.570796326794896558 -1.570796326794896558 0" />
@@ -230,5 +230,5 @@
       <origin xyz="5.3368019332749957491e-17 -0.29900000000000009903 -0.064999999999999974465" rpy="-5.5511151231257814695e-17 -0 3.141592653589793116" />
       <parent link="${prefix}base_link" />
-      <child link="${prefix}caster_wheel_link" />
+      <child link="${prefix}caster_wheel" />
       <axis xyz="0 0 1"/>
       <limit effort="1" velocity="20" />
@@ -236,5 +236,5 @@
     </joint>
     <!-- caster wheel Link -->
-    <link name="${prefix}caster_wheel_link">
+    <link name="${prefix}caster_wheel">
       <visual>
         <origin xyz="1.1302212892091925974e-17 5.5511151231257827021e-17 0" rpy="3.141592653589793116 -8.3802055560433424155e-17 -3.141592653589793116" />
