Commit message: update

File: urdf/diffbot_description.urdf.xacro (robot description, xacro)
@@ -59,5 +59,5 @@
     <!-- right wheel joint -->
     <joint name="${prefix}right_wheel_joint" type="continuous">
-      <origin xyz="-0.12500000000000002776 -2.7755575615628913511e-17 -0.060000000000000004718" rpy="-1.570796326794896558 -2.2204460492503130808e-16 -1.57079632679489678" />
+      <origin xyz="6.9388939039072283776e-17 -0.125 -0.05999999999999999778" rpy="-1.57079632679489678 -1.1660544913393859426e-16 6.9388939039072283776e-17" />
       <parent link="${prefix}base_link" />
       <child link="${prefix}right_wheel" />
@@ -91,5 +91,5 @@
     <!-- left wheel joint -->
     <joint name="${prefix}left_wheel_joint" type="continuous">
-      <origin xyz="0.125 1.3877787807814456755e-17 -0.05999999999999999778" rpy="1.57079632679489678 -1.1102230246251567869e-16 -1.570796326794896558" />
+      <origin xyz="-5.5511151231257827021e-17 0.12500000000000005551 -0.060000000000000011657" rpy="1.570796326794896558 -1.6964751660994284333e-16 1.7347234759768063549e-16" />
       <parent link="${prefix}base_link" />
       <child link="${prefix}left_wheel" />
@@ -123,5 +123,5 @@
     <!-- caster wheel joint -->
     <joint name="${prefix}caster_wheel_joint" type="fixed">
-      <origin xyz="-4.8640783256844265209e-17 0.29000000000000003553 -0.019999999999999990008" rpy="-5.5511151231257814695e-17 -0 3.141592653589793116" />
+      <origin xyz="-0.29000000000000003553 -1.236754434711827603e-16 -0.019999999999999969191" rpy="-5.5511151231257814695e-17 -0 3.141592653589793116" />
       <parent link="${prefix}base_link" />
       <child link="${prefix}caster_wheel" />
@@ -178,5 +178,5 @@
     <!-- laser_joint -->
     <joint name="${prefix}laser_joint" type="fixed">
-      <origin xyz="-2.778062350693125085e-18 -0.024999999999999994449 0.024999999999999997918" rpy="-3.141592653589793116 -6.1629758220391519929e-33 1.1102230246251560474e-16" />
+      <origin xyz="0.025000000000000001388 2.7755575615628913511e-17 0.025000000000000008327" rpy="-3.141592653589793116 -6.1629758220391519929e-33 1.1102230246251560474e-16" />
       <parent link="${prefix}base_link" />
       <child link="${prefix}laser_link" />
@@ -210,5 +210,5 @@
     <!-- Camera Joint -->
     <joint name="${prefix}camera_joint" type="fixed">
-      <origin xyz="-4.4452289071905681794e-18 -0.040000000000000007772 -1.3877787807814456755e-17" rpy="6.1062266354383530837e-16 1.1102230246251567869e-16 3.141592653589793116" />
+      <origin xyz="0.040000000000000007772 1.3877787807814456755e-17 -4.4408920985006270245e-18" rpy="6.1062266354383530837e-16 1.1102230246251567869e-16 3.141592653589793116" />
       <parent link="${prefix}base_link" />
       <child link="${prefix}camera_link" />

Commit message: update

File: urdf/diffbot_description.urdf.xacro (robot description, xacro)
@@ -58,5 +58,6 @@
     </joint>
     <!-- right wheel joint -->
-    <joint name="${prefix}right_wheel_joint" type="continuous">
+    <!-- fixed wheel joint for testing, type was continuous -->
+    <joint name="${prefix}right_wheel_joint" type="fixed">
       <origin xyz="6.9388939039072283776e-17 -0.125 -0.05999999999999999778" rpy="-1.57079632679489678 -1.1660544913393859426e-16 6.9388939039072283776e-17" />
       <parent link="${prefix}base_link" />
@@ -89,6 +90,7 @@
       </inertial>
     </link>
+    <!-- fixed wheel joint for testing, type was continuous -->
     <!-- left wheel joint -->
-    <joint name="${prefix}left_wheel_joint" type="continuous">
+    <joint name="${prefix}left_wheel_joint" type="fixed">
       <origin xyz="-5.5511151231257827021e-17 0.12500000000000005551 -0.060000000000000011657" rpy="1.570796326794896558 -1.6964751660994284333e-16 1.7347234759768063549e-16" />
       <parent link="${prefix}base_link" />

Commit message: update

File: urdf/diffbot_description.urdf.xacro (robot description, xacro)
@@ -19,5 +19,5 @@
     <xacro:property name="z_offset" value="-${base_height/2}" />
     <!-- Space btw top of beam and the each joint -->
-    <!-- dummy link - used for ros2 control so it stops complaining? -->
+    <!-- dummy link - used for ros2 control so it stops complaining?
     <link name="${prefix}dummy_link">
     </link>
@@ -25,5 +25,5 @@
       <parent link="${prefix}dummy_link" />
       <child link="${prefix}base_link" />
-    </joint>
+    </joint> -->
     <!-- needed for replacement to find mesh dir: file://$(find bot_mini_description)/mesh/ -->
     <!-- Base Link -->

Commit message: update

File: urdf/diffbot_description.urdf.xacro (robot description, xacro)
@@ -59,5 +59,5 @@
     <!-- right wheel joint -->
     <!-- fixed wheel joint for testing, type was continuous -->
-    <joint name="${prefix}right_wheel_joint" type="fixed">
+    <joint name="${prefix}right_wheel_joint" type="continuous">
       <origin xyz="6.9388939039072283776e-17 -0.125 -0.05999999999999999778" rpy="-1.57079632679489678 -1.1660544913393859426e-16 6.9388939039072283776e-17" />
       <parent link="${prefix}base_link" />
@@ -92,5 +92,5 @@
     <!-- fixed wheel joint for testing, type was continuous -->
     <!-- left wheel joint -->
-    <joint name="${prefix}left_wheel_joint" type="fixed">
+    <joint name="${prefix}left_wheel_joint" type="continuous">
       <origin xyz="-5.5511151231257827021e-17 0.12500000000000005551 -0.060000000000000011657" rpy="1.570796326794896558 -1.6964751660994284333e-16 1.7347234759768063549e-16" />
       <parent link="${prefix}base_link" />
