Commit message: update

File: urdf/diffbot_description.urdf.xacro (robot description, xacro)
@@ -18,5 +18,6 @@
     <xacro:property name="caster_wheel_radius" value="0.04" />
     <xacro:property name="z_offset" value="-${base_height/2}" />
-    <!-- Space btw top of beam and the each joint -->
+    <!-- Offset of main Axis to center of base body (Axis of rotation for steering) -->
+    <xacro:property name="base_offset" value="0.11" />
     <!-- dummy link - used for ros2 control so it stops complaining?
     <link name="${prefix}dummy_link">
@@ -45,5 +46,5 @@
       </collision>
       <inertial>
-        <origin xyz="-2.5368985414583082317e-17 0.083896718007622009261 -0.0037261823981863751235" rpy="0 0 0"/>
+        <origin xyz="0 0 0" rpy="0 0 0"/>
         <mass value="8.4123950268139715547" />
         <inertia ixx="0.090166990291185383777" ixy="4.7429179749238352248e-18" ixz="1.4209310488728267579e-18" iyy="0.055481261106946747064" iyz="-0.01112159061226025876" izz="0.13051099377067149065" />
@@ -61,5 +62,5 @@
     <!-- fixed wheel joint for testing, type was continuous -->
     <joint name="${prefix}right_wheel_joint" type="continuous">
-      <origin xyz="$(base_length/2) -0.125 ${z_offset}" rpy="0 0 0" />
+      <origin xyz="0 -0.125 ${z_offset}" rpy="0 0 0" />
       <parent link="${prefix}base_link" />
       <child link="${prefix}right_wheel" />
@@ -94,5 +95,5 @@
     <!-- left wheel joint -->
     <joint name="${prefix}left_wheel_joint" type="continuous">
-      <origin xyz="${(base_length/2)} 0.125 ${z_offset}" rpy="0 0 0" />
+      <origin xyz="0 0.125 ${z_offset}" rpy="0 0 0" />
       <parent link="${prefix}base_link" />
       <child link="${prefix}left_wheel" />
@@ -126,5 +127,5 @@
     <!-- caster wheel joint -->
     <joint name="${prefix}caster_wheel_joint" type="fixed">
-      <origin xyz="-${(base_length/2)} 0 -0.02" rpy="0 0 ${PI}" />
+      <origin xyz="-${base_length / 2 + base_offset} 0 -0.02" rpy="0 0 ${PI}" />
       <parent link="${prefix}base_link" />
       <child link="${prefix}caster_wheel" />
@@ -181,5 +182,5 @@
     <!-- laser_joint -->
     <joint name="${prefix}laser_joint" type="fixed">
-      <origin xyz="${(base_length/2)-0.035} 0 0" rpy="0 0 0"/>
+      <origin xyz="${base_length /2 -0.035 - base_offset} 0 0" rpy="0 0 0"/>
       <parent link="${prefix}base_link" />
       <child link="${prefix}laser_link" />
@@ -213,5 +214,5 @@
     <!-- Camera Joint -->
     <joint name="${prefix}camera_joint" type="fixed">
-      <origin xyz="${base_length/2} 0 0" rpy="0 0 ${PI}" />
+      <origin xyz="${base_length / 2 - base_offset} 0 0" rpy="0 0 ${PI}" />
       <parent link="${prefix}base_link" />
       <child link="${prefix}camera_link" />

Commit message: update

File: urdf/diffbot_description.urdf.xacro (robot description, xacro)
@@ -62,5 +62,5 @@
     <!-- fixed wheel joint for testing, type was continuous -->
     <joint name="${prefix}right_wheel_joint" type="continuous">
-      <origin xyz="0 -0.125 ${z_offset}" rpy="0 0 0" />
+      <origin xyz="0 -0.125 ${z_offset}" rpy="${PI} 0 0" />
       <parent link="${prefix}base_link" />
       <child link="${prefix}right_wheel" />
@@ -95,5 +95,5 @@
     <!-- left wheel joint -->
     <joint name="${prefix}left_wheel_joint" type="continuous">
-      <origin xyz="0 0.125 ${z_offset}" rpy="0 0 0" />
+      <origin xyz="0 0.125 ${z_offset}" rpy="${PI} 0 0" />
       <parent link="${prefix}base_link" />
       <child link="${prefix}left_wheel" />

Commit message: update

File: urdf/diffbot_description.urdf.xacro (robot description, xacro)
@@ -62,5 +62,5 @@
     <!-- fixed wheel joint for testing, type was continuous -->
     <joint name="${prefix}right_wheel_joint" type="continuous">
-      <origin xyz="0 -0.125 ${z_offset}" rpy="${PI} 0 0" />
+      <origin xyz="0 -0.125 ${z_offset}" rpy="${PI / 2} 0 0" />
       <parent link="${prefix}base_link" />
       <child link="${prefix}right_wheel" />
@@ -95,5 +95,5 @@
     <!-- left wheel joint -->
     <joint name="${prefix}left_wheel_joint" type="continuous">
-      <origin xyz="0 0.125 ${z_offset}" rpy="${PI} 0 0" />
+      <origin xyz="0 0.125 ${z_offset}" rpy="${PI / 2} 0 0" />
       <parent link="${prefix}base_link" />
       <child link="${prefix}left_wheel" />

Commit message: update

File: urdf/diffbot_description.urdf.xacro (robot description, xacro)
@@ -65,5 +65,5 @@
       <parent link="${prefix}base_link" />
       <child link="${prefix}right_wheel" />
-      <axis xyz="0 0 -1"/>
+      <axis xyz="0 0 1"/>
       <limit effort="1" velocity="20" />
       <joint_properties friction="0.0"/>

Commit message: update

File: urdf/diffbot_description.urdf.xacro (robot description, xacro)
@@ -27,5 +27,5 @@
       <child link="${prefix}base_link" />
     </joint> -->
-    <!-- needed for replacement to find mesh dir: file://$(find bot_mini_description)/mesh/ -->
+    <!-- needed for replacement to find mesh dir: package://bot_mini_description/mesh/ -->
     <!-- Base Link -->
     <link name="${prefix}base_link">
@@ -33,5 +33,5 @@
         <origin xyz="0 0 0" rpy="0 0 0" />
         <geometry>
-          <mesh filename="file://$(find bot_mini_description)/mesh/base_link_visual.stl"/>
+          <mesh filename="package://bot_mini_description/mesh/base_link_visual.stl"/>
         </geometry>
         <material name="base_link_material">
@@ -42,5 +42,5 @@
         <origin xyz="0 0 0" rpy="0 -0 0" />
         <geometry>
-          <mesh filename="file://$(find bot_mini_description)/mesh/base_link_collision.stl"/>
+          <mesh filename="package://bot_mini_description/mesh/base_link_collision.stl"/>
         </geometry>
       </collision>
@@ -74,5 +74,5 @@
         <origin xyz="0 0 0" rpy="0 -0 0" />
         <geometry>
-          <mesh filename="file://$(find bot_mini_description)/mesh/wheel_link_visual.stl"/>
+          <mesh filename="package://bot_mini_description/mesh/wheel_link_visual.stl"/>
         </geometry>
         <material name="wheel_link_material">
@@ -83,5 +83,5 @@
         <origin xyz="0 0 0" rpy="0 -0 0" />
         <geometry>
-          <mesh filename="file://$(find bot_mini_description)/mesh/wheel_link_collision.stl"/>
+          <mesh filename="package://bot_mini_description/mesh/wheel_link_collision.stl"/>
         </geometry>
       </collision>
@@ -107,5 +107,5 @@
         <origin xyz="0 0 0" rpy="0 -0 0" />
         <geometry>
-          <mesh filename="file://$(find bot_mini_description)/mesh/wheel_link_2_visual.stl"/>
+          <mesh filename="package://bot_mini_description/mesh/wheel_link_2_visual.stl"/>
         </geometry>
         <material name="wheel_link_2_material">
@@ -116,5 +116,5 @@
         <origin xyz="0 0 0" rpy="0 -0 0" />
         <geometry>
-          <mesh filename="file://$(find bot_mini_description)/mesh/wheel_link_2_collision.stl"/>
+          <mesh filename="package://bot_mini_description/mesh/wheel_link_2_collision.stl"/>
         </geometry>
       </collision>
@@ -139,5 +139,5 @@
         <origin xyz="0 0 0" rpy="0 -0 0" />
         <geometry>
-          <mesh filename="file://$(find bot_mini_description)/mesh/caster_link_visual.stl"/>
+          <mesh filename="package://bot_mini_description/mesh/caster_link_visual.stl"/>
         </geometry>
         <material name="caster_link_material">
@@ -148,5 +148,5 @@
         <origin xyz="0 0 0" rpy="0 -0 0" />
         <geometry>
-          <mesh filename="file://$(find bot_mini_description)/mesh/caster_link_collision.stl"/>
+          <mesh filename="package://bot_mini_description/mesh/caster_link_collision.stl"/>
         </geometry>
       </collision>
@@ -162,5 +162,5 @@
         <origin xyz="0 0 0" rpy="0 -0 0" />
         <geometry>
-          <mesh filename="file://$(find bot_mini_description)/mesh/laser_link_visual.stl"/>
+          <mesh filename="package://bot_mini_description/mesh/laser_link_visual.stl"/>
         </geometry>
         <material name="laser_link_material">
@@ -171,5 +171,5 @@
         <origin xyz="0 0 0" rpy="0 -0 0" />
         <geometry>
-          <mesh filename="file://$(find bot_mini_description)/mesh/laser_link_collision.stl"/>
+          <mesh filename="package://bot_mini_description/mesh/laser_link_collision.stl"/>
         </geometry>
       </collision>
@@ -194,5 +194,5 @@
         <origin xyz="0 0 0" rpy="0 -0 0" />
         <geometry>
-          <mesh filename="file://$(find bot_mini_description)/mesh/camera_link_visual.stl"/>
+          <mesh filename="package://bot_mini_description/mesh/camera_link_visual.stl"/>
         </geometry>
         <material name="camera_link_material">
@@ -203,5 +203,5 @@
         <origin xyz="0 0 0" rpy="0 -0 0" />
         <geometry>
-          <mesh filename="file://$(find bot_mini_description)/mesh/camera_link_collision.stl"/>
+          <mesh filename="package://bot_mini_description/mesh/camera_link_collision.stl"/>
         </geometry>
       </collision>

Commit message: update laser joint pos

File: urdf/diffbot_description.urdf.xacro (robot description, xacro)
@@ -182,5 +182,5 @@
     <!-- laser_joint -->
     <joint name="${prefix}laser_joint" type="fixed">
-      <origin xyz="${base_length /2 -0.035 - base_offset} 0 0" rpy="0 0 0"/>
+      <origin xyz="${base_length /2 -0.015 - base_offset} 0 0" rpy="0 0 0"/>
       <parent link="${prefix}base_link" />
       <child link="${prefix}laser_link" />

Commit message: update laser joint pos

File: urdf/diffbot_description.urdf.xacro (robot description, xacro)
@@ -182,5 +182,5 @@
     <!-- laser_joint -->
     <joint name="${prefix}laser_joint" type="fixed">
-      <origin xyz="${base_length /2 -0.015 - base_offset} 0 0" rpy="0 0 0"/>
+      <origin xyz="${base_length /2 +0.015 - base_offset} 0 -${z_offset}" rpy="0 0 0"/>
       <parent link="${prefix}base_link" />
       <child link="${prefix}laser_link" />

Commit message: update laser joint pos

File: urdf/diffbot_description.urdf.xacro (robot description, xacro)
@@ -182,5 +182,5 @@
     <!-- laser_joint -->
     <joint name="${prefix}laser_joint" type="fixed">
-      <origin xyz="${base_length /2 +0.015 - base_offset} 0 -${z_offset}" rpy="0 0 0"/>
+      <origin xyz="${base_length /2 +0.015 - base_offset} 0 ${z_offset * -1}" rpy="0 0 0"/>
       <parent link="${prefix}base_link" />
       <child link="${prefix}laser_link" />

Commit message: update laser joint pos

File: urdf/diffbot_description.urdf.xacro (robot description, xacro)
@@ -160,5 +160,5 @@
     <link name="${prefix}laser_link">
       <visual>
-        <origin xyz="0 0 0" rpy="0 -0 0" />
+        <origin xyz="0 0 0" rpy="180 -0 0" />
         <geometry>
           <mesh filename="package://bot_mini_description/mesh/laser_link_visual.stl"/>
@@ -169,5 +169,5 @@
       </visual>
       <collision>
-        <origin xyz="0 0 0" rpy="0 -0 0" />
+        <origin xyz="0 0 0" rpy="180 -0 0" />
         <geometry>
           <mesh filename="package://bot_mini_description/mesh/laser_link_collision.stl"/>
@@ -175,5 +175,5 @@
       </collision>
       <inertial>
-        <origin xyz="8.0502568807622093404e-21 2.7755575615628913511e-17 -0.01526549883836261258" rpy="0 0 0"/>
+        <origin xyz="8.0502568807622093404e-21 2.7755575615628913511e-17 -0.01526549883836261258" rpy="180 0 0"/>
         <mass value="0.065307030550339775776" />
         <inertia ixx="1.578111853789072904e-05" ixy="-4.8590457654361857326e-53" ixz="1.0816309858643350309e-52" iyy="1.5781118537890654501e-05" iyz="9.8088682514084147142e-38" izz="1.9760068210357054465e-05" />
@@ -182,5 +182,5 @@
     <!-- laser_joint -->
     <joint name="${prefix}laser_joint" type="fixed">
-      <origin xyz="${base_length /2 +0.015 - base_offset} 0 ${z_offset * -1}" rpy="0 0 0"/>
+      <origin xyz="${base_length /2 -0.015 - base_offset} 0 ${z_offset * -1 +0.05}" rpy="0 0 0"/>
       <parent link="${prefix}base_link" />
       <child link="${prefix}laser_link" />

Commit message: update laser joint pos

File: urdf/diffbot_description.urdf.xacro (robot description, xacro)
@@ -182,5 +182,5 @@
     <!-- laser_joint -->
     <joint name="${prefix}laser_joint" type="fixed">
-      <origin xyz="${base_length /2 -0.015 - base_offset} 0 ${z_offset * -1 +0.05}" rpy="0 0 0"/>
+      <origin xyz="-0.015 0 0.09" rpy="0 0 0"/>
       <parent link="${prefix}base_link" />
       <child link="${prefix}laser_link" />

Commit message: update laser joint pos

File: urdf/diffbot_description.urdf.xacro (robot description, xacro)
@@ -160,5 +160,5 @@
     <link name="${prefix}laser_link">
       <visual>
-        <origin xyz="0 0 0" rpy="180 -0 0" />
+        <origin xyz="0 0 0" rpy="${PI} -0 0" />
         <geometry>
           <mesh filename="package://bot_mini_description/mesh/laser_link_visual.stl"/>
@@ -169,5 +169,5 @@
       </visual>
       <collision>
-        <origin xyz="0 0 0" rpy="180 -0 0" />
+        <origin xyz="0 0 0" rpy="${PI} -0 0" />
         <geometry>
           <mesh filename="package://bot_mini_description/mesh/laser_link_collision.stl"/>
@@ -175,5 +175,5 @@
       </collision>
       <inertial>
-        <origin xyz="8.0502568807622093404e-21 2.7755575615628913511e-17 -0.01526549883836261258" rpy="180 0 0"/>
+        <origin xyz="8.0502568807622093404e-21 2.7755575615628913511e-17 -0.01526549883836261258" rpy="${PI} 0 0"/>
         <mass value="0.065307030550339775776" />
         <inertia ixx="1.578111853789072904e-05" ixy="-4.8590457654361857326e-53" ixz="1.0816309858643350309e-52" iyy="1.5781118537890654501e-05" iyz="9.8088682514084147142e-38" izz="1.9760068210357054465e-05" />

Commit message: update laser joint pos

File: urdf/diffbot_description.urdf.xacro (robot description, xacro)
@@ -62,8 +62,8 @@
     <!-- fixed wheel joint for testing, type was continuous -->
     <joint name="${prefix}right_wheel_joint" type="continuous">
-      <origin xyz="0 -0.125 ${z_offset}" rpy="${PI / 2} 0 0" />
+      <origin xyz="0 {-0.125 - wheel_len /2} ${z_offset}" rpy="${PI / 2} 0 0" />
       <parent link="${prefix}base_link" />
       <child link="${prefix}right_wheel" />
-      <axis xyz="0 0 1"/>
+      <axis xyz="0 0 -1"/>
       <limit effort="1" velocity="20" />
       <joint_properties friction="0.0"/>
@@ -72,5 +72,5 @@
     <link name="${prefix}right_wheel">
       <visual>
-        <origin xyz="0 0 0" rpy="0 -0 0" />
+        <origin xyz="0 -{wheel_len /2} 0" rpy="0 -0 0" />
         <geometry>
           <mesh filename="package://bot_mini_description/mesh/wheel_link_visual.stl"/>
@@ -95,8 +95,8 @@
     <!-- left wheel joint -->
     <joint name="${prefix}left_wheel_joint" type="continuous">
-      <origin xyz="0 0.125 ${z_offset}" rpy="${PI / 2} 0 0" />
+      <origin xyz="0 {0.125 + wheel_len /2} ${z_offset}" rpy="${PI / 2} 0 0" />
       <parent link="${prefix}base_link" />
       <child link="${prefix}left_wheel" />
-      <axis xyz="0 0 -1" />
+      <axis xyz="0 0 1" />
       <limit effort="1" velocity="20" />
       <joint_properties friction="0.0" />
@@ -105,5 +105,5 @@
     <link name="${prefix}left_wheel">
       <visual>
-        <origin xyz="0 0 0" rpy="0 -0 0" />
+        <origin xyz="0 {wheel_len /2} 0" rpy="0 -0 0" />
         <geometry>
           <mesh filename="package://bot_mini_description/mesh/wheel_link_2_visual.stl"/>
@@ -114,5 +114,5 @@
       </visual>
       <collision>
-        <origin xyz="0 0 0" rpy="0 -0 0" />
+        <origin xyz="0 {wheel_len /2} 0" rpy="0 -0 0" />
         <geometry>
           <mesh filename="package://bot_mini_description/mesh/wheel_link_2_collision.stl"/>

Commit message: update laser joint pos

File: urdf/diffbot_description.urdf.xacro (robot description, xacro)
@@ -62,5 +62,5 @@
     <!-- fixed wheel joint for testing, type was continuous -->
     <joint name="${prefix}right_wheel_joint" type="continuous">
-      <origin xyz="0 {-0.125 - wheel_len /2} ${z_offset}" rpy="${PI / 2} 0 0" />
+      <origin xyz="0 ${-0.125 - wheel_len /2} ${z_offset}" rpy="${PI / 2} 0 0" />
       <parent link="${prefix}base_link" />
       <child link="${prefix}right_wheel" />
@@ -72,5 +72,5 @@
     <link name="${prefix}right_wheel">
       <visual>
-        <origin xyz="0 -{wheel_len /2} 0" rpy="0 -0 0" />
+        <origin xyz="0 -${wheel_len /2} 0" rpy="0 -0 0" />
         <geometry>
           <mesh filename="package://bot_mini_description/mesh/wheel_link_visual.stl"/>
@@ -81,5 +81,5 @@
       </visual>
       <collision>
-        <origin xyz="0 0 0" rpy="0 -0 0" />
+        <origin xyz="0 -${wheel_len /2} 0" rpy="0 -0 0" />
         <geometry>
           <mesh filename="package://bot_mini_description/mesh/wheel_link_collision.stl"/>
@@ -95,5 +95,5 @@
     <!-- left wheel joint -->
     <joint name="${prefix}left_wheel_joint" type="continuous">
-      <origin xyz="0 {0.125 + wheel_len /2} ${z_offset}" rpy="${PI / 2} 0 0" />
+      <origin xyz="0 ${0.125 + wheel_len /2} ${z_offset}" rpy="${PI / 2} 0 0" />
       <parent link="${prefix}base_link" />
       <child link="${prefix}left_wheel" />
@@ -105,5 +105,5 @@
     <link name="${prefix}left_wheel">
       <visual>
-        <origin xyz="0 {wheel_len /2} 0" rpy="0 -0 0" />
+        <origin xyz="0 ${wheel_len /2} 0" rpy="0 -0 0" />
         <geometry>
           <mesh filename="package://bot_mini_description/mesh/wheel_link_2_visual.stl"/>
@@ -114,5 +114,5 @@
       </visual>
       <collision>
-        <origin xyz="0 {wheel_len /2} 0" rpy="0 -0 0" />
+        <origin xyz="0 ${wheel_len /2} 0" rpy="0 -0 0" />
         <geometry>
           <mesh filename="package://bot_mini_description/mesh/wheel_link_2_collision.stl"/>

Commit message: update laser joint pos

File: urdf/diffbot_description.urdf.xacro (robot description, xacro)
@@ -72,5 +72,5 @@
     <link name="${prefix}right_wheel">
       <visual>
-        <origin xyz="0 -${wheel_len /2} 0" rpy="0 -0 0" />
+        <origin xyz="0 0 ${wheel_len}" rpy="0 -0 0" />
         <geometry>
           <mesh filename="package://bot_mini_description/mesh/wheel_link_visual.stl"/>
@@ -81,5 +81,5 @@
       </visual>
       <collision>
-        <origin xyz="0 -${wheel_len /2} 0" rpy="0 -0 0" />
+        <origin xyz="0 0 ${wheel_len}" rpy="0 -0 0" />
         <geometry>
           <mesh filename="package://bot_mini_description/mesh/wheel_link_collision.stl"/>
@@ -105,5 +105,5 @@
     <link name="${prefix}left_wheel">
       <visual>
-        <origin xyz="0 ${wheel_len /2} 0" rpy="0 -0 0" />
+        <origin xyz="0 0 ${wheel_len}" rpy="0 -0 0" />
         <geometry>
           <mesh filename="package://bot_mini_description/mesh/wheel_link_2_visual.stl"/>
@@ -114,5 +114,5 @@
       </visual>
       <collision>
-        <origin xyz="0 ${wheel_len /2} 0" rpy="0 -0 0" />
+        <origin xyz="0 0 ${wheel_len}" rpy="0 -0 0" />
         <geometry>
           <mesh filename="package://bot_mini_description/mesh/wheel_link_2_collision.stl"/>

Commit message: added imu link joint

File: urdf/diffbot_description.urdf.xacro (robot description, xacro)
@@ -221,4 +221,25 @@
       <joint_properties friction="0.0"/>
     </joint>
+    <!-- imu_link -->
+    <link name="${prefix}imu_link">
+      <visual>
+        <origin xyz="0 0 0" rpy="0 -0 0" />
+      </visual>
+      <collision>
+        <origin xyz="0 0 0" rpy="0 -0 0" />
+      </collision>
+      <inertial>
+        <origin xyz="5.3378961738576549005e-07 0.0016484827975361887251 -0.020840554768345870285" rpy="0 0 0"/>
+      </inertial>
+    </link>
+    <!-- imu Joint -->
+    <joint name="${prefix}imu_joint" type="fixed">
+      <origin xyz="${base_length / 2 - base_offset} 0 0" rpy="0 0 ${PI}" />
+      <parent link="${prefix}base_link" />
+      <child link="${prefix}imu_link" />
+      <axis xyz="0 0 1"/>
+      <limit effort="1" velocity="20" />
+      <joint_properties friction="0.0"/>
+    </joint>
   </xacro:macro>
 </robot>
