Commit message: update

File: urdf/diffbot_description.urdf.xacro (robot description, xacro)
@@ -144,5 +144,5 @@
         <parent link="${prefix}chassis"/>
         <child link="${prefix}laser_frame"/>
-        <origin xyz="-0.07 0 0.10" rpy="0 0 ${pi}"/>
+        <origin xyz="${chassis_length/2 -0.07} 0 0.10" rpy="0 0 ${pi}"/>
     </joint>
     <link name="${prefix}laser_frame">

Commit message: update

File: urdf/diffbot_description.urdf.xacro (robot description, xacro)
@@ -14,5 +14,5 @@
     <xacro:property name="wheel_mass" value="0.02"/>
     <xacro:property name="wheel_offset_x" value="0.285748"/>
-    <xacro:property name="wheel_offset_y" value="0.33675"/>
+    <xacro:property name="wheel_offset_y" value="0.13"/>
     <xacro:property name="wheel_offset_z" value="-0.035"/>
     <xacro:property name="caster_wheel_radius" value="0.04"/>
@@ -91,5 +91,5 @@
         <parent link="${prefix}chassis"/>
         <child link="${prefix}left_wheel"/>
-        <origin xyz="${chassis_length/2 - 0.075} ${wheel_offset_y/2 + wheel_thickness/2 + 0.01} ${wheel_offset_z}" rpy="-${pi/2} 0 0" />
+        <origin xyz="${chassis_length/2 - chassis_offset} ${wheel_offset_y/2 + wheel_thickness/2 + 0.01} ${wheel_offset_z}" rpy="-${pi/2} 0 0" />
         <axis xyz="0 0 1"/>
     </joint>

Commit message: update

File: urdf/diffbot_description.urdf.xacro (robot description, xacro)
@@ -63,5 +63,5 @@
         <parent link="${prefix}chassis"/>
         <child link="${prefix}right_wheel"/>
-        <origin xyz="${chassis_length/2 - 0.075} -${wheel_offset_y/2 + wheel_thickness/2 + 0.01} ${wheel_offset_z}" rpy="${pi/2} 0 0" />
+        <origin xyz="${chassis_length/2 - 0.075} -${wheel_offset_y + wheel_thickness/2 + 0.01} ${wheel_offset_z}" rpy="${pi/2} 0 0" />
         <axis xyz="0 0 -1"/>
         <limit effort="1" velocity="20" />
@@ -91,5 +91,5 @@
         <parent link="${prefix}chassis"/>
         <child link="${prefix}left_wheel"/>
-        <origin xyz="${chassis_length/2 - chassis_offset} ${wheel_offset_y/2 + wheel_thickness/2 + 0.01} ${wheel_offset_z}" rpy="-${pi/2} 0 0" />
+        <origin xyz="${chassis_length/2 - chassis_offset} ${wheel_offset_y + wheel_thickness/2 + 0.01} ${wheel_offset_z}" rpy="-${pi/2} 0 0" />
         <axis xyz="0 0 1"/>
     </joint>

Commit message: update

File: urdf/diffbot_description.urdf.xacro (robot description, xacro)
@@ -60,5 +60,5 @@
     </gazebo>
     <!-- RIGHT WHEEL -->
-    <joint name="${prefix}right_wheel_joint" type="continuous">
+    <joint name="${prefix}right_wheel_joint" type="fixed">
         <parent link="${prefix}chassis"/>
         <child link="${prefix}right_wheel"/>
@@ -88,5 +88,5 @@
     </gazebo>
     <!-- LEFT WHEEL -->
-    <joint name="${prefix}left_wheel_joint" type="continuous">
+    <joint name="${prefix}left_wheel_joint" type="fixed">
         <parent link="${prefix}chassis"/>
         <child link="${prefix}left_wheel"/>

Commit message: update

File: urdf/diffbot_description.urdf.xacro (robot description, xacro)
@@ -63,5 +63,5 @@
         <parent link="${prefix}chassis"/>
         <child link="${prefix}right_wheel"/>
-        <origin xyz="${chassis_length/2 - 0.075} -${wheel_offset_y + wheel_thickness/2 + 0.01} ${wheel_offset_z}" rpy="${pi/2} 0 0" />
+        <origin xyz="${chassis_length/2 - 0.075} -${wheel_offset_y + wheel_thickness/2} ${wheel_offset_z}" rpy="${pi/2} 0 0" />
         <axis xyz="0 0 -1"/>
         <limit effort="1" velocity="20" />
@@ -91,5 +91,5 @@
         <parent link="${prefix}chassis"/>
         <child link="${prefix}left_wheel"/>
-        <origin xyz="${chassis_length/2 - chassis_offset} ${wheel_offset_y + wheel_thickness/2 + 0.01} ${wheel_offset_z}" rpy="-${pi/2} 0 0" />
+        <origin xyz="${chassis_length/2 - chassis_offset} ${wheel_offset_y + wheel_thickness/2} ${wheel_offset_z}" rpy="-${pi/2} 0 0" />
         <axis xyz="0 0 1"/>
     </joint>

Commit message: update

File: urdf/diffbot_description.urdf.xacro (robot description, xacro)
@@ -144,5 +144,5 @@
         <parent link="${prefix}chassis"/>
         <child link="${prefix}laser_frame"/>
-        <origin xyz="${chassis_length/2 -0.07} 0 0.10" rpy="0 0 ${pi}"/>
+        <origin xyz="${chassis_length/2 -0.07} 0 0.10" rpy="0 0 0"/>
     </joint>
     <link name="${prefix}laser_frame">

Commit message: update: remounted laser

File: urdf/diffbot_description.urdf.xacro (robot description, xacro)
@@ -141,8 +141,9 @@
     </gazebo>
     <!-- LASER -->
+    <!-- now rotated and mounted on the underside -->
     <joint name="${prefix}laser_joint" type="fixed">
         <parent link="${prefix}chassis"/>
         <child link="${prefix}laser_frame"/>
-        <origin xyz="${chassis_length/2 -0.07} 0 0.10" rpy="0 0 0"/>
+        <origin xyz="${chassis_length/2 -chassis_offset} 0 -0.07" rpy="${2*pi} 0 0"/>
     </joint>
     <link name="${prefix}laser_frame">

Commit message: update

File: urdf/diffbot_description.urdf.xacro (robot description, xacro)
@@ -145,5 +145,5 @@
         <parent link="${prefix}chassis"/>
         <child link="${prefix}laser_frame"/>
-        <origin xyz="${chassis_length/2 -chassis_offset} 0 -0.07" rpy="${2*pi} 0 0"/>
+        <origin xyz="${chassis_length/2 -chassis_offset} 0 -0.07" rpy="${pi} 0 0"/>
     </joint>
     <link name="${prefix}laser_frame">
